File: Node/NodeHardware/MCU_And_Peripherals.kicad_sch (KiCad schematic)
At the start: 35 parts, among them SW1 RST, SW2 BTN, U6 UCC27511ADBV, U7 ESP32-S3-WROOM-1

Commit message: Finish all the basic SCHM needed for the ESP32
Parts:
- removed JP9: SolderJumper_2_Bridged, Jumper:SolderJumper-2_P1.3mm_Bridged2Bar_RoundedPad1.0x1.5mm, symbol Jumper:SolderJumper_2_Bridged
- removed R15, R18, R25: R, Resistor_SMD:R_0805_2012Metric, symbol Device:R
- removed TP11, TP12: TestPoint, TestPoint:TestPoint_Pad_D2.0mm, symbol Connector:TestPoint_Alt
- added C13: C, Capacitor_SMD:C_0805_2012Metric, symbol Device:C
- added C21: 100n, Capacitor_SMD:C_0805_2012Metric, symbol Device:C
- added Q3, Q4: 2N7002, Package_TO_SOT_SMD:SOT-23, symbol Transistor_FET:2N7002
- added R12, R37: 2k2, Resistor_SMD:R_0805_2012Metric, symbol Device:R
- added R34, R35: 0R, Resistor_SMD:R_0805_2012Metric, symbol Device:R
- added R36, R38, R39: 10k, Resistor_SMD:R_0805_2012Metric, symbol Device:R
- added SW3: BOOT, symbol Switch:SW_Push
- C14: value C -> 1u
- C15, C18: value C -> 100n
- D10, D11, D5, D8, D9: value LED -> YELLOW
- D6: value LED -> RED
- D7: value LED -> GREEN
- R13, R14, R16: value R -> 47k
- R17, R19, R20, R21, R22, R23, R24: value R -> 2k2
Connections:
- net +BATT: now also R14.1; no longer R13.1
- net GND: now also C16.2, C17.2, C18.2, R20.2, R21.2, SW1.2, SW2.2, C13.2, C21.2, SW3.2; no longer C16.1
- net I2C_SDA: now also R22.2
- net SPI_MISO: now also R17.2
- net SPI_MOSI: now also R12.2
- net UART_UC_RX: now also R23.2, U7.36 (U0RXD/GPIO44/CLK_OUT2)
- net UART_UC_TX: now also R24.2, U7.37 (U0TXD/GPIO43/CLK_OUT1)
- net LED_01: now reaches TP9.1
- net LED_01: now also D6.2 (A)
- net BATT_SENSE: now reaches R14.2
- net BATT_SENSE: now also C18.1, R16.1; no longer TH1.1
- net PCB_TEMP: now reaches R13.2
- net PCB_TEMP: now also TH1.1, C21.1; no longer R16.1
- net I2C_SDA_LED_K: now reaches R22.1
- net I2C_SDA_LED_K: now also D9.1 (K)
- net SPI_MISO_LED_K: now reaches D8.1 (K)
- net SPI_MISO_LED_K: now also R17.1
- net +3V3: now reaches D8.2 (A)
- net +3V3: now also C14.2, C15.2, D10.2 (A), D11.2 (A), D5.2 (A), D9.2 (A), R13.1, U7.2 (3V3), R36.1, R38.1, R39.1
- net LED_01_K: now reaches R20.1
- net LED_01_K: now also D6.1 (K)
- net JTAG_RST: now reaches SW1.1
- net JTAG_RST: now also U7.3 (EN), C13.1, Q3.3 (D), R38.2
- net SPI_MOSI_LED_K: now reaches D5.1 (K)
- net SPI_MOSI_LED_K: now also R12.1
- net UART_TX_LED_K: now reaches R24.1
- net UART_TX_LED_K: now also D11.1 (K)
- net at U7.13 (GPIO19/U1RTS/ADC2_CH8/CLK_OUT2/USB_D-): now also R34.2
- net at U7.14 (GPIO20/U1CTS/ADC2_CH9/CLK_OUT1/USB_D+): now also R35.2
- net BOOT: now reaches U7.27 (GPIO0/BOOT)
- net BOOT: now also C16.1, Q4.3 (D), R39.2, SW3.1
- net JTAG_TCK: now reaches U7.32 (MTCK/GPIO39/CLK_OUT3/SUBSPICS1)
- net JTAG_TDO: now reaches U7.33 (MTDO/GPIO40/CLK_OUT2)
- net JTAG_TDI: now reaches U7.34 (MTDI/GPIO41/CLK_OUT1)
- net JTAG_TMS: now reaches U7.35 (MTMS/GPIO42)
- net USER_BUTTON: now reaches SW2.1
- net USER_BUTTON: now also C17.1, R36.2
- net CH340_DTR: now reaches R19.1
- net CH340_DTR: now also Q4.2 (S)
- net at R19.2: now also Q3.1 (G)
- net LED_02_K: now reaches D7.1 (K)
- net LED_02_K: now also R21.1
- net LED_02: now reaches D7.2 (A)
- net LED_02: now also TP10.1
- net UART_RX_LED_K: now reaches D10.1 (K)
- net UART_RX_LED_K: now also R23.1
- removed net +3.3V: C14.2, C15.2, C16.2, R14.1, U7.2 (3V3)
- new net: Q4.1 (G), R37.2
- new net CH340_RTS: Q3.2 (S), R37.1
- new net USB_D+: R35.1
- new net USB_D-: R34.1
Other:
- note added: "Blinky LED"
- note added: "Boot mode select button"
- note added: "CH340 USB TO UART RST/BOOT CONTROL"
- note added: "I2C activity LED"
- note added: "Reset button"
- note added: "Status LEDs"
- note added: "TODO: check if I2C is active low???"
- note added: "TODO: check if SPI is active low???"
- note added: "TODO: check if UART is active low???"
- note added: "User button"
- note added: "WiFi status"
- note removed: "I2C activity LEDs"
- note removed: "Mini debug - blinky"
- note removed: "WiFi connection status"
- moved on the sheet: C14, C15, C17, SW2, TH1, U6, U7

Commit message: Finish first version of inputs
Parts:
- added C24, C25, C27, C28, C29, C30, C31, C32, C33, C34: 100n, Capacitor_SMD:C_0805_2012Metric, symbol Device:C
- added D13, D14, D15, D17, D19, D20, D21, D22, D24, D26, D27, D28: SS34, Diode_SMD:D_SMA, symbol Diode:SS34
- added D16, D18, D23, D25: 3V6, Diode_SMD:D_SOD-123, symbol Device:D_Zener
- added R45, R47, R53, R55, R57, R59: 100R, Resistor_SMD:R_0805_2012Metric, symbol Device:R
- added R46, R48, R54, R56, R58, R60: 10k, Resistor_SMD:R_0805_2012Metric, symbol Device:R
- added R50, R52, R63, R64: 220k, Resistor_SMD:R_0805_2012Metric, symbol Device:R
- added R61, R62, R65, R66: 100k, Resistor_SMD:R_0805_2012Metric, symbol Device:R
- TH1: value PCB_TEMP_NTC -> 10k
- renumbered C14 to C17, C15 to C18, C13 to C19, C16 to C20, C17 to C21, C18 to C22, C21 to C23, D5 to D10, D8 to D11, D9 to D12, D10 to D8, D11 to D9, R35 to R28, R34 to R29, R20 to R30, R21 to R31, R23 to R32, R24 to R33, R12 to R34, R17 to R35, R22 to R36, R19 to R37, R36 to R40, R37 to R41, R14 to R42, R13 to R43, R16 to R44, SW3 to SW2, SW2 to SW3, U7 to U6, U6 to U7
Connections:
- net +3V3: now also D13.1 (K), D15.1 (K), D17.1 (K), D20.1 (K), D21.1 (K), D26.1 (K)
- net GND: now also C24.2, C25.2, C27.2, C28.2, C29.2, C30.2, C31.2, C32.2, C33.2, C34.2, D14.2 (A), D16.2 (A), D18.2 (A), D19.2 (A), D22.2 (A), D23.2 (A), D24.2 (A), D25.2 (A), D27.2 (A), D28.2 (A), R46.2, R48.2, R54.2, R56.2, R58.2, R60.2, R61.2, R62.2, R65.2, R66.2
- new net ANA_IN_01: R50.1
- new net ANA_IN_01_UC: C27.1, D16.1 (K), R50.2, R61.1
- new net ANA_IN_02: R52.1
- new net ANA_IN_02_UC: C32.1, D18.1 (K), R52.2, R62.1
- new net ANA_IN_03: R64.1
- new net ANA_IN_03_UC: C34.1, D25.1 (K), R64.2, R66.1
- new net ANA_IN_04: R63.1
- new net ANA_IN_04_UC: C33.1, D23.1 (K), R63.2, R65.1
- new net DIG_IO_01: R57.2
- new net DIG_IO_01_UC: C30.1, D21.2 (A), D22.1 (K), R57.1, R58.1
- new net DIG_IO_02: R53.2
- new net DIG_IO_02_UC: C28.1, D17.2 (A), D19.1 (K), R53.1, R54.1
- new net DIG_IO_03: R55.2
- new net DIG_IO_03_UC: C29.1, D20.2 (A), D24.1 (K), R55.1, R56.1
- new net DIG_IO_04: R59.2
- new net DIG_IO_04_UC: C31.1, D26.2 (A), D28.1 (K), R59.1, R60.1
- new net DIG_IO_05: R45.2
- new net DIG_IO_05_UC: C24.1, D13.2 (A), D14.1 (K), R45.1, R46.1
- new net DIG_IO_06: R47.2
- new net DIG_IO_06_UC: C25.1, D15.2 (A), D27.1 (K), R47.1, R48.1
Other:
- note added: "Analog inputs"
- note added: "Digital I/O"
- note added: "If needed, use output shift registers or some precision ADC input IC"
- note added: "Open drain and PWM outputs"
- note added: "Overvoltage prot. Rev. pol. prot."
- note added: "TODO: think about adding 5v, 3v3 and 3v3LP voltage sense"
- note removed: "INPUTS"
- note removed: "If needed, use ADC input multiplexer, or external analog input IC"
- note removed: "If needed, use output shift registers"
- note removed: "OUTPUTS"
- moved on the sheet: C22, C23, R42, R43, R44, TH1, U7

Commit message: Add a comment
Other:
- note added: "TODO: change diodes to a double diode package with smaller footprint"
Changed lines of the file:
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@@
+		)
+	)
+	(text "TODO:\nchange diodes to a double diode package\nwith smaller footprint"
+		(exclude_from_sim no)
+		(at 269.494 246.126 0)
+		(effects
+			(font
+				(size 2.4 2.4)
+			)
 		)
 	)
