File: Node/NodeHardware/MCU_And_Peripherals.kicad_sch (KiCad schematic)
At the start: 108 parts, among them Q4 2N7002, Q5 2N7002, SW1 RST, SW2 BOOT, SW3 BTN, U10 UCC27517DBVR, U11 IRLR024NTRPBF, U4 ADS1220xPW, U6 UCC27517DBVR, U7 ESP32-S3-WROOM-1, U8 IRLR024NTRPBF

Commit message: Never ending SCHM design
Parts:
- removed C28, C33, C34, C9: 100n, Capacitor_SMD:C_0805_2012Metric, symbol Device:C
- removed D15, D16, D17, D18, D19, D20, D24, D25, D26, D27, D28, D29: SS34, Diode_SMD:D_SMA, symbol Diode:SS34
- removed R11, R12: 47k, Resistor_SMD:R_0805_2012Metric, symbol Device:R
- removed R43, R59, R60, R67, R68: 10k, Resistor_SMD:R_0805_2012Metric, symbol Device:R
- removed R61, R70: ???, Resistor_SMD:R_0805_2012Metric, symbol Device:R
- removed R64, R65: 100R, Resistor_SMD:R_0805_2012Metric, symbol Device:R
- removed U10, U6: UCC27517DBVR, UCC27517DBVR:UCC27517DBVR_DBV5_TEX, symbol UCC27517DBVR:UCC27517DBVR
- removed U11, U8: IRLR024NTRPBF, IRLR024NTRPBF:IRLR024NTRPBF_PG-TO252-3_INF, symbol IRLR024NTRPBF:IRLR024NTRPBF
- added C16, C17, C20, C21, C25, C36: 100n, Capacitor_SMD:C_0805_2012Metric, symbol Device:C
- added D10, D5, D6, D7, D8, D9: BAT54S, Package_TO_SOT_SMD:SOT-23, symbol Diode:BAT54S
- added Q3, Q4: AO3400A, Package_TO_SOT_SMD:SOT-23, symbol Transistor_FET:AO3400A
- added R24, R25, R30, R31, R38, R73: 10k, Resistor_SMD:R_0805_2012Metric, symbol Device:R
- added R26, R27, R32, R33: 220R, Resistor_SMD:R_0805_2012Metric, symbol Device:R
- added R28, R29, R34, R35, R40: 100R, Resistor_SMD:R_0805_2012Metric, symbol Device:R
- added R48, R49, R50, R51, R52: 47R, Resistor_SMD:R_0805_2012Metric, symbol Device:R
- added U7: ADS1220xPW, Package_SO:TSSOP-16_4.4x5mm_P0.65mm, symbol Analog_ADC:ADS1220xPW
- C18: renamed from C17; value 1u -> 22u
- C22: value C -> 100n
- C28: renamed from C20; value C -> 1u
- R53, R54, R55: value 100R -> 47R
- R58: value 10k -> 2k2
- renumbered C18 to C19, C35 to C23, C19 to C24, C23 to C26, C10 to C30, C21 to C31, C25 to C32, C32 to C33, C8 to C34, C11 to C35, C26 to C37, C31 to C38, C24 to C39, D6 to D11, D7 to D12, D8 to D13, D9 to D14, D5 to D15, D21 to D16, D13 to D17, D23 to D18, D10 to D19, D11 to D20, D14 to D21, D12 to D23, Q4 to Q5, Q5 to Q6, R29 to R36, R32 to R37, R69 to R39, R66 to R41, R33 to R42, R34 to R43, R40 to R44, R44 to R45, R35 to R46, R36 to R47, R41 to R56, R26 to R57, R28 to R59, R42 to R60, R30 to R61, R31 to R62, R37 to R63, R38 to R64, R48 to R65, R50 to R66, R56 to R67, R63 to R68, R9 to R69, R10 to R70, R45 to R71, R47 to R72, R39 to R74, R49 to R75, R51 to R76, R52 to R77, R62 to R78, R46 to R79, U7 to U6, U4 to U8
Connections:
- net 3V3_SENSE is gone; now on net ANA_IN_01_UC: U8.11 (AIN0/REFP1)
- net +3V3: now also C27.2, SW3.2, C25.2, D10.2 (K), D5.2 (K), D6.2 (K), D7.2 (K), D8.2 (K), D9.2 (K), U7.12 (AVDD), U7.13 (DVDD)
- net 5V_SENSE: now also U7.10 (AIN1); no longer U8.10 (AIN1)
- net ANA_IN_01_UC: no longer U6.38 (GPIO2/TOUCH2/ADC1_CH1)
- net ANA_IN_02_UC: now also U8.10 (AIN1); no longer U6.15 (GPIO3/TOUCH3/ADC1_CH2)
- net ANA_IN_03_UC: now also U8.7 (AIN2); no longer U6.4 (GPIO4/TOUCH4/ADC1_CH3)
- net ANA_IN_04_UC: now also U8.6 (AIN3/REFN1); no longer U6.5 (GPIO5/TOUCH5/ADC1_CH4)
- net BATT_SENSE: now also U7.7 (AIN2); no longer U8.7 (AIN2)
- net DIG_IO_01: now also R28.2; no longer R53.2
- net DIG_IO_01_UC: now also U6.20 (GPIO12/TOUCH12/ADC2_CH1/FSPICLK/FSPIIO6/SUBSPICLK), C16.1, D5.3 (COM), R24.1, R28.1; no longer C27.1, R53.1, R58.1
- net DIG_IO_02: now also R34.2; no longer R54.2
- net DIG_IO_02_UC: now also U6.21 (GPIO13/TOUCH13/ADC2_CH2/FSPIQ/FSPIIO7/SUBSPIQ), C20.1, D7.3 (COM), R30.1, R34.1; no longer R54.1
- net DIG_IO_03: now also R40.2; no longer R55.2
- net DIG_IO_03_UC: now also C22.1, U6.22 (GPIO14/TOUCH14/ADC2_CH3/FSPIWP/FSPIDQS/SUBSPIWP), D9.3 (COM), R38.1, R40.1; no longer C29.1, R55.1
- net DIG_IO_04: now also R29.2
- net DIG_IO_04_UC: now also U6.23 (GPIO21), C17.1, D6.3 (COM), R25.1, R29.1
- net DIG_IO_05: now also R35.2
- net DIG_IO_05_UC: now also U6.31 (GPIO38/FSPIWP/SUBSPIWP), C21.1, D8.3 (COM), R31.1, R35.1
- net DIG_IO_06_UC: now also U6.24 (GPIO47/SPICLK_P/SUBSPICLK_P_DIFF), D10.3 (COM)
- net DIG_OUT_01: now also Q3.3 (D)
- net DIG_OUT_01_UC: now also U6.4 (GPIO4/TOUCH4/ADC1_CH3), R26.1
- net DIG_OUT_02: now also Q4.3 (D)
- net DIG_OUT_02_UC: now also U6.5 (GPIO5/TOUCH5/ADC1_CH4), R32.1
- net GND: now also C27.1, C16.2, C17.2, C20.2, C21.2, C25.1, C36.2, D10.1 (A), D5.1 (A), D6.1 (A), D7.1 (A), D8.1 (A), D9.1 (A), Q3.2 (S), Q4.2 (S), R24.2, R25.2, R27.2, R30.2, R31.2, R33.2, R38.2, R73.2, U7.3 (CLK), U7.4 (DGND), U7.5 (AVSS); no longer C27.2, R58.2, SW3.2
- net I2C_SCL: now also U6.39 (GPIO1/TOUCH1/ADC1_CH0)
- net I2C_SDA: now also U6.38 (GPIO2/TOUCH2/ADC1_CH1)
- net JTAG_RST: now also R58.1; no longer SW1.1
- net LED_01: now also U6.26 (GPIO45)
- net LED_02: now also U6.16 (GPIO46)
- net PCB_TEMP: now also U7.11 (AIN0/REFP1); no longer U6.39 (GPIO1/TOUCH1/ADC1_CH0)
- net PWR_SENSE: now also U7.6 (AIN3/REFN1); no longer U8.6 (AIN3/REFN1)
- net SPI_MISO: now also R54.2, U6.30 (SPIDQS/GPIO37/FSPIQ/SUBSPIQ), R50.2; no longer U8.15 (DOUT/~{DRDY})
- net SPI_MOSI: now also R53.2, U6.28 (SPIIO6/GPIO35/FSPID/SUBSPID), R49.2; no longer U8.16 (DIN)
- net SPI_SCLK: now also U6.29 (SPIIO7/GPIO36/FSPICLK/SUBSPICLK), R48.2, R52.2; no longer U8.1 (SCLK)
- net USER_BUTTON: now also U6.15 (GPIO3/TOUCH3/ADC1_CH2), C36.1, R73.1; no longer C22.1
- net SPI_CS_EXT: now reaches U6.25 (GPIO48/SPICLK_N/SUBSPICLK_N_DIFF)
- net SPI_CS_ADC0: now reaches U6.8 (GPIO15/U0RTS/ADC2_CH4/XTAL_32K_P)
- net SPI_CS_ADC0: now also R51.2
- net SPI_CS_ADC1: now reaches U6.9 (GPIO16/U0CTS/ADC2_CH5/XTAL_32K_N)
- net SPI_CS_ADC1: now also R55.2
- net SPI_CS_ADC: no longer names the net of U8.2 (~{CS})
- net SPI_CS_ADC: now also R55.1
- new net: R49.1, U7.16 (DIN)
- new net: C29.1, R58.2, SW1.1
- new net: Q3.1 (G), R26.2, R27.1
- new net: R48.1, U7.1 (SCLK)
- new net: R50.1, U7.15 (DOUT/~{DRDY})
- new net: R51.1, U7.2 (~{CS})
- new net: R52.1, U8.1 (SCLK)
- new net: R54.1, U8.15 (DOUT/~{DRDY})
- new net: R53.1, U8.16 (DIN)
- new net: Q4.1 (G), R32.2, R33.1
- no-connect marks 10 -> 12
Other:
- note added: "*bootstrap"
- note added: "ADC - analog inputs"
- note added: "ADC - on-board sensors"
- note added: "AO3400A N MOSFET"
- note added: "BAT54S Dual diode package UV/OV prot."
- note removed: "ADC1 CH0-CH4"
- note removed: "DIG IN/OUT"
- note removed: "IRLR024NTRPBF N MOSFET"
- note removed: "Overvoltage prot. Rev. pol. prot."
- note removed: "UCC27517DBVR Low side gate driver, open drain output"
- moved on the sheet: C23, C24, C26, C28, C30, C34, C35, R39, R41, R56, R61, R62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

Commit message: Halfway working on PCB for Node
Parts:
- removed C26, C27: 100n, Capacitor_SMD:C_0805_2012Metric, symbol Device:C
- removed TP10, TP9: TestPoint, TestPoint:TestPoint_Pad_D2.0mm, symbol Connector:TestPoint_Alt
- added D24, D25, D26, D27: YELLOW, LED_SMD:LED_1210_3225Metric, symbol Device:LED
- added R80: 10k, Resistor_SMD:R_0805_2012Metric, symbol Device:R
- added TP14: TP_UART0_RX, TestPoint:TestPoint_Pad_D1.0mm, symbol Connector:TestPoint_Small
- added TP15: TP_UART0_TX, TestPoint:TestPoint_Pad_D1.0mm, symbol Connector:TestPoint_Small
- added TP16: TP_I2C_SCL, TestPoint:TestPoint_Pad_D1.0mm, symbol Connector:TestPoint_Small
- added TP17: TP_I2C_SDA, TestPoint:TestPoint_Pad_D1.0mm, symbol Connector:TestPoint_Small
- added TP18: TP_DIGOUT_01, TestPoint:TestPoint_Pad_D1.0mm, symbol Connector:TestPoint_Small
- added TP19: TP_DIGOUT_02, TestPoint:TestPoint_Pad_D1.0mm, symbol Connector:TestPoint_Small
- added TP20: TP_SPI_CS_0, TestPoint:TestPoint_Pad_D1.0mm, symbol Connector:TestPoint_Small
- added TP21: TP_SPI_CS_1, TestPoint:TestPoint_Pad_D1.0mm, symbol Connector:TestPoint_Small
- added TP22: TP_SPI_MOSI, TestPoint:TestPoint_Pad_D1.0mm, symbol Connector:TestPoint_Small
- added TP23: TP_SPI_SCLK, TestPoint:TestPoint_Pad_D1.0mm, symbol Connector:TestPoint_Small
- added TP24: TP_SPI_MISO, TestPoint:TestPoint_Pad_D1.0mm, symbol Connector:TestPoint_Small
- added TP25: TP_SPI_CS_EXT, TestPoint:TestPoint_Pad_D1.0mm, symbol Connector:TestPoint_Small
- added TP26, TP58: TP_DIG_IO_06, TestPoint:TestPoint_Pad_D1.0mm, symbol Connector:TestPoint_Small
- added TP27, TP56: TP_DIG_IO_05, TestPoint:TestPoint_Pad_D1.0mm, symbol Connector:TestPoint_Small
- added TP28, TP52: TP_DIG_IO_04, TestPoint:TestPoint_Pad_D1.0mm, symbol Connector:TestPoint_Small
- added TP29, TP57: TP_DIG_IO_03, TestPoint:TestPoint_Pad_D1.0mm, symbol Connector:TestPoint_Small
- added TP30, TP55: TP_DIG_IO_02, TestPoint:TestPoint_Pad_D1.0mm, symbol Connector:TestPoint_Small
- added TP31, TP54: TP_DIG_IO_01, TestPoint:TestPoint_Pad_D1.0mm, symbol Connector:TestPoint_Small
- added TP32: TP_UART1_TX, TestPoint:TestPoint_Pad_D1.0mm, symbol Connector:TestPoint_Small
- added TP33: TP_UART1_RX, TestPoint:TestPoint_Pad_D1.0mm, symbol Connector:TestPoint_Small
- added TP34: TP_GPIO6, TestPoint:TestPoint_Pad_D1.0mm, symbol Connector:TestPoint_Small
- added TP35: TP_GPIO7, TestPoint:TestPoint_Pad_D1.0mm, symbol Connector:TestPoint_Small
- added TP36: TP_GPIO8, TestPoint:TestPoint_Pad_D1.0mm, symbol Connector:TestPoint_Small
- added TP37: TP_GPIO9, TestPoint:TestPoint_Pad_D1.0mm, symbol Connector:TestPoint_Small
- added TP38: TP_GPIO10, TestPoint:TestPoint_Pad_D1.0mm, symbol Connector:TestPoint_Small
- added TP39: TP_GPIO11, TestPoint:TestPoint_Pad_D1.0mm, symbol Connector:TestPoint_Small
- added TP40: TP_ANA_IN_01_UC, TestPoint:TestPoint_Pad_D1.0mm, symbol Connector:TestPoint_Small
- added TP41: TP_ANA_IN_01, TestPoint:TestPoint_Pad_D1.0mm, symbol Connector:TestPoint_Small
- added TP42: TP_ANA_IN_02_UC, TestPoint:TestPoint_Pad_D1.0mm, symbol Connector:TestPoint_Small
- added TP43: TP_ANA_IN_02, TestPoint:TestPoint_Pad_D1.0mm, symbol Connector:TestPoint_Small
- added TP44: TP_ANA_IN_04_UC, TestPoint:TestPoint_Pad_D1.0mm, symbol Connector:TestPoint_Small
- added TP45: TP_ANA_IN_04, TestPoint:TestPoint_Pad_D1.0mm, symbol Connector:TestPoint_Small
- added TP46: TP_ANA_IN_03_UC, TestPoint:TestPoint_Pad_D1.0mm, symbol Connector:TestPoint_Small
- added TP47: TP_ANA_IN_03, TestPoint:TestPoint_Pad_D1.0mm, symbol Connector:TestPoint_Small
- added TP49: TP_DIG_OUT_01, TestPoint:TestPoint_Pad_D1.0mm, symbol Connector:TestPoint_Small
- added TP51: TP_DIG_OUT_02, TestPoint:TestPoint_Pad_D1.0mm, symbol Connector:TestPoint_Small
- R63: value 10kk -> 10k
- SW1, SW2, SW3: footprint (none) -> Button_Switch_SMD:SW_Push_1P1T_NO_6x6mm_H9.5mm
Connections:
- net +3V3: now also D24.2 (A)
- net ANA_IN_01: now also TP41.1
- net ANA_IN_01_UC: now also TP40.1
- net ANA_IN_02: now also TP43.1
- net ANA_IN_02_UC: now also TP42.1
- net ANA_IN_03: now also TP47.1
- net ANA_IN_03_UC: now also TP46.1
- net ANA_IN_04: now also TP45.1
- net ANA_IN_04_UC: now also TP44.1
- net DIG_IO_01: now also TP54.1
- net DIG_IO_01_UC: now also TP31.1
- net DIG_IO_02: now also TP55.1
- net DIG_IO_02_UC: now also TP30.1
- net DIG_IO_03: now also TP57.1
- net DIG_IO_03_UC: now also TP29.1
- net DIG_IO_04: now also TP52.1
- net DIG_IO_04_UC: now also TP28.1
- net DIG_IO_05: now also TP56.1
- net DIG_IO_05_UC: now also TP27.1
- net DIG_IO_06: now also TP58.1
- net DIG_IO_06_UC: now also TP26.1
- net DIG_OUT_01: now also TP49.1
- net DIG_OUT_01_UC: now also TP18.1
- net DIG_OUT_02: now also TP51.1
- net DIG_OUT_02_UC: now also TP19.1
- net GND: now also D25.1 (K), D26.1 (K), D27.1 (K)
- net I2C_SCL: now also TP16.1
- net I2C_SDA: now also TP17.1
- net SPI_CS_ADC0: now also R64.2, TP20.1
- net SPI_CS_ADC1: now also R63.2, TP21.1
- net SPI_CS_EXT: now also R80.2, TP25.1
- net SPI_MISO: now also TP24.1; no longer R64.2
- net SPI_MOSI: now also TP22.1; no longer R63.2
- net SPI_SCLK: now also TP23.1
- net UART0_UC_RX: now also TP14.1
- net UART0_UC_TX: now also TP15.1
- net UART1_UC_RX: now also TP33.1
- net UART1_UC_TX: now also TP32.1
- net at U6.12 (GPIO8/TOUCH8/ADC1_CH7/SUBSPICS1): now also TP36.1
- net at U6.17 (GPIO9/TOUCH9/ADC1_CH8/FSPIHD/SUBSPIHD): now also TP37.1
- net at U6.18 (GPIO10/TOUCH10/ADC1_CH9/FSPICS0/FSPIIO4/SUBSPICS0): now also TP38.1
- net at U6.19 (GPIO11/TOUCH11/ADC2_CH0/FSPID/FSPIIO5/SUBSPID): now also TP39.1
- net at U6.6 (GPIO6/TOUCH6/ADC1_CH5): now also TP34.1
- net at U6.7 (GPIO7/TOUCH7/ADC1_CH6): now also TP35.1
- net JTAG_RST renamed RST
- net SPI_MISO_LED_K renamed SPI_CS_LED_0_K
- net SPI_CS_LED_0_K: now also D27.2 (A)
- net SPI_MOSI_LED_K renamed SPI_CS_LED_1_K
- net SPI_CS_LED_1_K: now also D26.2 (A)
- new net SPI_CS_LED_EXT_K: D24.1 (K), D25.2 (A), R80.1
- no-connect marks 12 -> 6
Other:
- note added: "Decoupling cap"
- moved on the sheet: D11, D12, D13, D14, D15, D16, D19, D20, D23, Q3, Q4, R26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

Commit message: Continue updating PCB (main form)
Parts:
- removed C22, C23: 100n, Capacitor_SMD:C_0805_2012Metric, symbol Device:C
- removed D10, D9: BAT54S, Package_TO_SOT_SMD:SOT-23, symbol Diode:BAT54S
- removed R38, R39: 10k, Resistor_SMD:R_0805_2012Metric, symbol Device:R
- removed R40, R41: 100R, Resistor_SMD:R_0805_2012Metric, symbol Device:R
- removed TP57: TP_DIG_IO_03, TestPoint:TestPoint_Pad_D1.0mm, symbol Connector:TestPoint_Small
- removed TP58: TP_DIG_IO_06, TestPoint:TestPoint_Pad_D1.0mm, symbol Connector:TestPoint_Small
- added TP33: TP_GPIO45, TestPoint:TestPoint_Pad_D1.0mm, symbol Connector:TestPoint_Small
- added TP35: TP_GPIO46, TestPoint:TestPoint_Pad_D1.0mm, symbol Connector:TestPoint_Small
- renumbered C18 to C16, C19 to C17, C28 to C18, C29 to C19, C31 to C20, C36 to C21, C25 to C22, C30 to C23, C34 to C24, C35 to C25, C39 to C26, C32 to C27, C37 to C28, C24 to C29, C16 to C30, C20 to C31, C38 to C32, C17 to C34, C21 to C35, D15 to D10, D16 to D11, D23 to D12, D11 to D13, D12 to D14, D25 to D15, D26 to D16, D27 to D17, D17 to D18, D21 to D19, D5 to D20, D7 to D21, D18 to D23, D6 to D24, D8 to D25, D24 to D5, D19 to D6, D20 to D7, D13 to D8, D14 to D9, Q5 to Q3, Q6 to Q4, Q3 to Q5, Q4 to Q6, R46 to R24, R47 to R25, R57 to R26, R59 to R27, R74 to R28, R42 to R29, R43 to R30, R64 to R31, R36 to R32, R63 to R33, R37 to R34, R80 to R35, R44 to R36, R56 to R37, R60 to R38, R58 to R39, R73 to R40, R45 to R41, R61 to R42, R69 to R43, R71 to R44, R79 to R45, R62 to R46, R70 to R47, R72 to R48, R48 to R49, R26 to R50, R32 to R51, R49 to R52, R50 to R53, R27 to R54, R33 to R55, R51 to R56, R65 to R57, R75 to R58, R66 to R59, R76 to R60, R77 to R61, R67 to R62, R28 to R63, R34 to R64, R24 to R65, R30 to R66, R78 to R67, R52 to R69, R53 to R70, R54 to R71, R55 to R72, R29 to R73, R35 to R74, R25 to R75, R31 to R76, TP15 to TP12, TP14 to TP13, TP20 to TP14, TP21 to TP15, TP34 to TP20, TP35 to TP21, TP36 to TP22, TP37 to TP23, TP38 to TP24, TP39 to TP25, TP31 to TP26, TP30 to TP27, TP29 to TP28, TP32 to TP29, TP33 to TP30, TP28 to TP31, TP27 to TP32, TP22 to TP34, TP23 to TP36, TP26 to TP37, TP24 to TP38, TP25 to TP39, TP49 to TP40, TP51 to TP41, TP41 to TP42, TP40 to TP44, TP42 to TP45, TP45 to TP46, TP54 to TP48, TP55 to TP49, TP44 to TP50, TP46 to TP51, TP56 to TP53
Connections:
- net DIG_IO_05 is gone; now on net DIG_IO_04: R74.2, TP53.1
- net DIG_IO_06_UC is gone; now on net LED_02: TP37.1, U6.24 (GPIO47/SPICLK_P/SUBSPICLK_P_DIFF)
- net DIG_IO_03: now also R73.2, TP52.1
- net DIG_IO_03_UC: now also C34.1, D24.3 (COM), R73.1, R75.1
- net DIG_IO_04: no longer R73.2, TP52.1
- net DIG_IO_04_UC: now also C35.1, D25.3 (COM), R74.1, R76.1; no longer C34.1, D24.3 (COM), R73.1, R75.1
- net LED_01: now also TP32.1, U6.31 (GPIO38/FSPIWP/SUBSPIWP); no longer U6.26 (GPIO45)
- net LED_02: no longer U6.16 (GPIO46)
- removed net DIG_IO_05_UC: C35.1, D25.3 (COM), R74.1, R76.1, TP32.1, U6.31 (GPIO38/FSPIWP/SUBSPIWP)
- new net: TP35.1, U6.16 (GPIO46)
- new net: TP33.1, U6.26 (GPIO45)
Other:
- moved on the sheet: C30, C31, C34, C35, D20, D21, D24, D25, R63, R64, R65, R66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
