File: Node/NodeHardware/NodeHardware.kicad_pcb (KiCad board)
At the start: 2 copper layers, 100 x 100 mm, 87 parts, among them J1 USB_C_Receptacle_16P, Q1 AO3401A, Q2 AO3401A, U1 TPS565201DDCR, U2 TPS565201DDCR, U3 CH340C, U4 TLV70433DBVR, U5 MCP73831-2-OT, U6 UCC27511ADBV, U7 ESP32-S3-WROOM-1

Commit message: Add a comment
Parts:
- removed JP9: SolderJumper_2_Bridged, Jumper:SolderJumper-2_P1.3mm_Bridged2Bar_RoundedPad1.0x1.5mm
- removed TP11, TP12: TestPoint, TestPoint:TestPoint_Pad_D2.0mm
- added C12: 100n, Capacitor_SMD:C_0805_2012Metric, F.Cu at (185.5, 89.8)
- added C13: 4u7, Capacitor_SMD:C_0805_2012Metric, F.Cu at (185.5, 92.8)
- added C21: C, Capacitor_SMD:C_0805_2012Metric, F.Cu at (130.7, 72.1)
- added C22: 100n, Capacitor_SMD:C_0805_2012Metric, F.Cu at (130.7, 75.1)
- added C23: 100n, Capacitor_SMD:C_0805_2012Metric, F.Cu at (135.2, 60.1)
- added C24: 100n, Capacitor_SMD:C_0805_2012Metric, F.Cu at (135.2, 63.1)
- added C25: 100n, Capacitor_SMD:C_0805_2012Metric, F.Cu at (135.2, 66.1)
- added C27: 100n, Capacitor_SMD:C_0805_2012Metric, F.Cu at (135.2, 69.1)
- added C28: 100n, Capacitor_SMD:C_0805_2012Metric, F.Cu at (135.2, 72.1)
- added C29: 100n, Capacitor_SMD:C_0805_2012Metric, F.Cu at (135.2, 75.1)
- added C30: 100n, Capacitor_SMD:C_0805_2012Metric, F.Cu at (139.6, 60.1)
- added C31: 100n, Capacitor_SMD:C_0805_2012Metric, F.Cu at (139.6, 63.1)
- added C32: 100n, Capacitor_SMD:C_0805_2012Metric, F.Cu at (139.6, 66.1)
- added C33: 100n, Capacitor_SMD:C_0805_2012Metric, F.Cu at (139.6, 69.1)
- added C34: 100n, Capacitor_SMD:C_0805_2012Metric, F.Cu at (139.6, 72.1)
- added D12: YELLOW, LED_SMD:LED_1210_3225Metric, F.Cu at (149.8, 104.7)
- added D13: SS34, Diode_SMD:D_SMA, F.Cu at (108.3, 60.9)
- added D14: SS34, Diode_SMD:D_SMA, F.Cu at (108.3, 65.4)
- added D15: SS34, Diode_SMD:D_SMA, F.Cu at (108.3, 70.0)
- added D16: 3V6, Diode_SMD:D_SOD-123, F.Cu at (144.8, 60.2)
- added D17: SS34, Diode_SMD:D_SMA, F.Cu at (108.3, 74.5)
- added D18: 3V6, Diode_SMD:D_SOD-123, F.Cu at (144.8, 63.6)
- added D19: SS34, Diode_SMD:D_SMA, F.Cu at (116.4, 60.9)
- added D20: SS34, Diode_SMD:D_SMA, F.Cu at (116.4, 65.4)
- added D21: SS34, Diode_SMD:D_SMA, F.Cu at (116.4, 70.0)
- added D22: SS34, Diode_SMD:D_SMA, F.Cu at (116.4, 74.5)
- added D23: 3V6, Diode_SMD:D_SOD-123, F.Cu at (144.8, 67.0)
- added D24: SS34, Diode_SMD:D_SMA, F.Cu at (124.5, 60.9)
- added D25: 3V6, Diode_SMD:D_SOD-123, F.Cu at (144.8, 70.3)
- added D26: SS34, Diode_SMD:D_SMA, F.Cu at (124.5, 65.4)
- added D27: SS34, Diode_SMD:D_SMA, F.Cu at (124.5, 70.0)
- added D28: SS34, Diode_SMD:D_SMA, F.Cu at (124.5, 74.5)
- added Q3: 2N7002, Package_TO_SOT_SMD:SOT-23, F.Cu at (150.1, 61.0)
- added Q4: 2N7002, Package_TO_SOT_SMD:SOT-23, F.Cu at (150.1, 65.6)
- added R34: 2k2, Resistor_SMD:R_0805_2012Metric, F.Cu at (106.4, 96.0)
- added R35: 2k2, Resistor_SMD:R_0805_2012Metric, F.Cu at (106.4, 98.9)
- added R36: 2k2, Resistor_SMD:R_0805_2012Metric, F.Cu at (110.8, 78.2)
- added R37: 2k2, Resistor_SMD:R_0805_2012Metric, F.Cu at (110.8, 81.2)
- added R38: 10k, Resistor_SMD:R_0805_2012Metric, F.Cu at (110.8, 84.2)
- added R39: 10k, Resistor_SMD:R_0805_2012Metric, F.Cu at (110.8, 87.1)
- added R40: 10k, Resistor_SMD:R_0805_2012Metric, F.Cu at (110.8, 90.0)
- added R41: 2k2, Resistor_SMD:R_0805_2012Metric, F.Cu at (110.8, 93.0)
- added R42: 47k, Resistor_SMD:R_0805_2012Metric, F.Cu at (110.8, 96.0)
- added R43: 47k, Resistor_SMD:R_0805_2012Metric, F.Cu at (110.8, 98.9)
- added R44: 47k, Resistor_SMD:R_0805_2012Metric, F.Cu at (115.3, 78.2)
- added R45: 100R, Resistor_SMD:R_0805_2012Metric, F.Cu at (115.3, 81.2)
- added R46: 10k, Resistor_SMD:R_0805_2012Metric, F.Cu at (115.3, 84.2)
- added R47: 100R, Resistor_SMD:R_0805_2012Metric, F.Cu at (115.3, 87.1)
- added R48: 10k, Resistor_SMD:R_0805_2012Metric, F.Cu at (115.3, 90.0)
- added R50: 220k, Resistor_SMD:R_0805_2012Metric, F.Cu at (115.3, 93.0)
- added R52: 220k, Resistor_SMD:R_0805_2012Metric, F.Cu at (115.3, 96.0)
- added R53: 100R, Resistor_SMD:R_0805_2012Metric, F.Cu at (115.3, 98.9)
- added R54: 10k, Resistor_SMD:R_0805_2012Metric, F.Cu at (119.7, 78.2)
- added R55: 100R, Resistor_SMD:R_0805_2012Metric, F.Cu at (119.7, 81.2)
- added R56: 10k, Resistor_SMD:R_0805_2012Metric, F.Cu at (119.7, 84.2)
- added R57: 100R, Resistor_SMD:R_0805_2012Metric, F.Cu at (119.7, 87.1)
- added R58: 10k, Resistor_SMD:R_0805_2012Metric, F.Cu at (119.7, 90.0)
- added R59: 100R, Resistor_SMD:R_0805_2012Metric, F.Cu at (119.7, 93.0)
- added R60: 10k, Resistor_SMD:R_0805_2012Metric, F.Cu at (119.7, 96.0)
- added R61: 100k, Resistor_SMD:R_0805_2012Metric, F.Cu at (119.7, 98.9)
- added R62: 100k, Resistor_SMD:R_0805_2012Metric, F.Cu at (124.1, 78.2)
- added R63: 220k, Resistor_SMD:R_0805_2012Metric, F.Cu at (124.1, 81.2)
- added R64: 220k, Resistor_SMD:R_0805_2012Metric, F.Cu at (124.1, 84.2)
- added R65: 100k, Resistor_SMD:R_0805_2012Metric, F.Cu at (124.1, 87.1)
- added R66: 100k, Resistor_SMD:R_0805_2012Metric, F.Cu at (124.1, 90.0)
- C14, C17: value C -> 1u
- C15, C18: value C -> 100n
- C16: value C -> 4u7
- C19: value 1u -> C
- C20: value 100n -> C
- D10, D11, D8, D9: value LED -> YELLOW
- D4: value 5V1 -> BLUE; footprint Diode_SMD:D_SOD-123 -> LED_SMD:LED_1210_3225Metric
- D5: value LED -> 5V1; footprint LED_SMD:LED_1210_3225Metric -> Diode_SMD:D_SOD-123
- D6: value LED -> RED
- D7: value LED -> GREEN
- R1, R29: value 10k -> 0R
- R10: value 5k1 -> ???
- R11: value 5k1 -> INF
- R12: value 47k -> 4k7
- R13, R14, R17, R19, R20, R21, R22, R24, R8: value 47k -> 0R
- R15: value 47k -> 10k
- R16, R18: value 47k -> 5k1
- R2: value 54.9k -> 10k
- R23: value 47k -> 2k2
- R26: value 0R -> 47k
- R27: value 4k7 -> 47k
- R3: value 0R -> 54.9k
- R30, R31, R32, R33: value 0R -> 2k2
- R4: value 10k -> INF
- R6: value ??? -> 4k7
- R7: value 4k7 -> 10k
- TH1: value PCB_TEMP_NTC -> 10k
- TP1: value 5V_TP -> V_IN_TP
- TP2: value V_IN_TP -> 5V_TP
- TP8: value TestPoint -> 3V3_LP_TP
- U6: value UCC27511ADBV -> ESP32-S3-WROOM-1; footprint Package_TO_SOT_SMD:SOT-23-6 -> Espressif:ESP32-S3-WROOM-1
- U7: value ESP32-S3-WROOM-1 -> UCC27511ADBV; footprint Espressif:ESP32-S3-WROOM-1 -> Package_TO_SOT_SMD:SOT-23-6
- moved J1 63.1 mm to (186.1, 64.0)
- moved R28 60.8 mm to (106.4, 78.2)
- moved U5 59.6 mm to (181.4, 96.7)
- moved R31 58.7 mm to (106.4, 87.1)
- moved R29 58.7 mm to (106.4, 81.2)
- moved R30 58.7 mm to (106.4, 84.2)
- moved R32 58.7 mm to (106.4, 90.0)
- moved R33 58.7 mm to (106.4, 93.0)
- moved U1 48.6 mm to (187.4, 70.8)
- moved U2 48.6 mm to (187.4, 75.2)
- moved Q1 48.6 mm to (182.7, 71.1)
- moved Q2 48.6 mm to (182.7, 75.7)
- moved U4 47.9 mm to (186.2, 96.5)
- moved R8 46.9 mm to (169.2, 60.0)
- moved R10 46.9 mm to (169.2, 66.0)
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Connections:
- C10 pad 1: +3.3V -> +3V3
- C10 pad 2: PWR_IN_N -> BATT_N
- C11 pad 1: +3.3V -> +3V3
- C11 pad 2: PWR_IN_N -> BATT_N
- C14 pad 1: PWR_IN_N -> +3V3_LP
- C14 pad 2: +3.3V -> BATT_N
- C15 pad 1: PWR_IN_N -> +BATT
- C15 pad 2: +3.3V -> BATT_N
- C16 pad 1: PWR_IN_N -> BATT_P
- C16 pad 2: +3.3V -> BATT_N
- C17 pad 1: unconnected-(C17-Pad1) -> BATT_N
- C17 pad 2: unconnected-(C17-Pad2) -> +3V3
- C18 pad 1: unconnected-(C18-Pad1) -> BATT_N
- C18 pad 2: unconnected-(C18-Pad2) -> +3V3
- C19 pad 1: unconnected-(C19-Pad1) -> JTAG_RST
- C19 pad 2: unconnected-(C19-Pad2) -> BATT_N
- C20 pad 1: unconnected-(C20-Pad1) -> BOOT
- C20 pad 2: unconnected-(C20-Pad2) -> BATT_N
- C3 pad 1: +5V -> V_IN
- C3 pad 2: PWR_IN_N -> BATT_N
- C4 pad 1: +5V -> V_IN
- C4 pad 2: PWR_IN_N -> BATT_N
- C6 pad 1: V_IN -> +5V
- C6 pad 2: PWR_IN_N -> BATT_N
- C7 pad 1: V_IN -> +5V
- C7 pad 2: PWR_IN_N -> BATT_N
- D10 pad 1: unconnected-(D10-K-Pad1) -> /MCU_And_Peripherals/SPI_MOSI_LED_K
- D10 pad 2: unconnected-(D10-A-Pad2) -> +3V3
- D11 pad 1: unconnected-(D11-K-Pad1) -> /MCU_And_Peripherals/SPI_MISO_LED_K
- D11 pad 2: unconnected-(D11-A-Pad2) -> +3V3
- D3 pad 2: +3.3V -> +3V3
- D4 pad 1: unconnected-(D4-K-Pad1) -> /BATT_LED_K
- D4 pad 2: unconnected-(D4-A-Pad2) -> Net-(D4-A)
- D5 pad 1: unconnected-(D5-K-Pad1) -> +BATT
- D5 pad 2: unconnected-(D5-A-Pad2) -> /BATT_IN_ZENER
- D6 pad 1: unconnected-(D6-K-Pad1) -> /MCU_And_Peripherals/LED_01_K
- D6 pad 2: unconnected-(D6-A-Pad2) -> LED_01
- D7 pad 1: unconnected-(D7-K-Pad1) -> /MCU_And_Peripherals/LED_02_K
- D7 pad 2: unconnected-(D7-A-Pad2) -> LED_02
- D8 pad 1: unconnected-(D8-K-Pad1) -> /MCU_And_Peripherals/UART_RX_LED_K
- D8 pad 2: unconnected-(D8-A-Pad2) -> +3V3
- D9 pad 1: unconnected-(D9-K-Pad1) -> /MCU_And_Peripherals/UART_TX_LED_K
- D9 pad 2: unconnected-(D9-A-Pad2) -> +3V3
- H1 pad 1: PWR_IN_N -> BATT_N
- H2 pad 1: PWR_IN_N -> BATT_N
- H3 pad 1: PWR_IN_N -> BATT_N
- H4 pad 1: PWR_IN_N -> BATT_N
- J1 pad A1: PWR_IN_N -> BATT_N
- J1 pad A12: PWR_IN_N -> BATT_N
- J1 pad B1: PWR_IN_N -> BATT_N
- J1 pad B12: PWR_IN_N -> BATT_N
- Q2 pad 1: unconnected-(Q2-G-Pad1) -> /BATT_IN_ZENER
- Q2 pad 2: unconnected-(Q2-S-Pad2) -> +BATT
- Q2 pad 3: unconnected-(Q2-D-Pad3) -> BATT_P
- R1 pad 1: /5V_REG_IN -> V_IN
- R1 pad 2: 5V_REG_EN -> /5V_REG_IN
- R10 pad 1: Net-(J1-CC1) -> +3V3
- R10 pad 2: PWR_IN_N -> /3V3_REG_VFB
- R11 pad 1: Net-(J1-CC2) -> BATT_N
- R11 pad 2: PWR_IN_N -> 3V3_REG_EN
- R12 pad 1: unconnected-(R12-Pad1) -> /3V3_REG_LED_K
- R12 pad 2: unconnected-(R12-Pad2) -> BATT_N
- R13 pad 1: +3.3V -> +3V3
- R13 pad 2: Net-(R13-Pad2) -> Net-(U3-V3)
- R14 pad 1: +BATT -> VBUS
- R14 pad 2: Net-(R14-Pad2) -> +5V
- R15 pad 1: unconnected-(R15-Pad1) -> /3V3_REG_VFB
- R15 pad 2: unconnected-(R15-Pad2) -> BATT_N
- R16 pad 1: Net-(R14-Pad2) -> Net-(J1-CC1)
- R16 pad 2: PWR_IN_N -> BATT_N
- R17 pad 1: unconnected-(R17-Pad1) -> /net_lable
- R17 pad 2: unconnected-(R17-Pad2) -> UART_UC_RX
- R18 pad 1: unconnected-(R18-Pad1) -> Net-(J1-CC2)
- R18 pad 2: unconnected-(R18-Pad2) -> BATT_N
- R19 pad 1: unconnected-(R19-Pad1) -> /net_lable
- R19 pad 2: unconnected-(R19-Pad2) -> UART_UC_TX
- R2 pad 1: +5V -> /5V_REG_IN
- R2 pad 2: /5V_REG_VFB -> 5V_REG_EN
- R20 pad 1: unconnected-(R20-Pad1) -> USB_D+
- R20 pad 2: unconnected-(R20-Pad2) -> /CH340_USB_D+
- R21 pad 1: unconnected-(R21-Pad1) -> USB_D-
- R21 pad 2: unconnected-(R21-Pad2) -> /CH340_USB_D-
- R22 pad 1: unconnected-(R22-Pad1) -> Net-(D4-A)
- R22 pad 2: unconnected-(R22-Pad2) -> +5V
- R23 pad 1: unconnected-(R23-Pad1) -> Net-(U5-STAT)
- R23 pad 2: unconnected-(R23-Pad2) -> /BATT_LED_K
- R24 pad 1: unconnected-(R24-Pad1) -> +BATT
- R24 pad 2: unconnected-(R24-Pad2) -> /3V3_LP_REG_IN
- R25 pad 1: +5V -> Net-(U5-PROG)
- R25 pad 2: /3V3_REG_IN -> Net-(R25-Pad2)
- R26 pad 1: V_IN -> /BATT_IN_ZENER
- R26 pad 2: /5V_REG_IN -> BATT_N
- R27 pad 1: /5V_REG_LED_K -> Net-(R25-Pad2)
- R27 pad 2: PWR_IN_N -> BATT_N
- R28 pad 1: unconnected-(R28-Pad1) -> USB_D+
- R28 pad 2: unconnected-(R28-Pad2) -> Net-(U6-GPIO20/U1CTS/ADC2_CH9/CLK_OUT1/USB_D+)
- R29 pad 1: /3V3_REG_IN -> USB_D-
- R29 pad 2: 3V3_REG_EN -> Net-(U6-GPIO19/U1RTS/ADC2_CH8/CLK_OUT2/USB_D-)
- R3 pad 1: VBUS -> +5V
- R3 pad 2: +5V -> /5V_REG_VFB
- R30 pad 1: USB_D+ -> /MCU_And_Peripherals/LED_01_K
- R30 pad 2: /CH340_USB_D+ -> BATT_N
- R31 pad 1: USB_D- -> /MCU_And_Peripherals/LED_02_K
- R31 pad 2: /CH340_USB_D- -> BATT_N
- R32 pad 1: unconnected-(R32-Pad1) -> /MCU_And_Peripherals/UART_RX_LED_K
- R32 pad 2: unconnected-(R32-Pad2) -> UART_UC_RX
- R33 pad 1: unconnected-(R33-Pad1) -> /MCU_And_Peripherals/UART_TX_LED_K
- R33 pad 2: unconnected-(R33-Pad2) -> UART_UC_TX
- R4 pad 1: /5V_REG_VFB -> BATT_N
- R4 pad 2: PWR_IN_N -> 5V_REG_EN
- R5 pad 2: PWR_IN_N -> BATT_N
- R6 pad 1: +3.3V -> /5V_REG_LED_K
- R6 pad 2: /3V3_REG_VFB -> BATT_N
- R7 pad 1: /3V3_REG_LED_K -> /5V_REG_VFB
- R7 pad 2: PWR_IN_N -> BATT_N
- R8 pad 1: unconnected-(R8-Pad1) -> +5V
- R8 pad 2: unconnected-(R8-Pad2) -> /3V3_REG_IN
- R9 pad 1: /3V3_REG_VFB -> /3V3_REG_IN
- R9 pad 2: PWR_IN_N -> 3V3_REG_EN
- TH1 pad 1: Net-(R13-Pad2) -> PCB_TEMP
- TH1 pad 2: PWR_IN_N -> BATT_N
- TP1 pad 1: +5V -> V_IN
- TP10 pad 1: unconnected-(TP10-Pad1) -> LED_02
- TP2 pad 1: V_IN -> +5V
- TP3 pad 1: PWR_IN_N -> BATT_N
- TP4 pad 1: PWR_IN_N -> BATT_N
- TP5 pad 1: PWR_IN_N -> BATT_N
- TP6 pad 1: PWR_IN_N -> BATT_N
- TP7 pad 1: +3.3V -> +3V3
- TP8 pad 1: unconnected-(TP8-Pad1) -> +3V3_LP
- TP9 pad 1: unconnected-(TP9-Pad1) -> LED_01
- U1 pad 1: PWR_IN_N -> BATT_N
- U2 pad 1: PWR_IN_N -> BATT_N
- U3 pad 1: PWR_IN_N -> BATT_N
- U3 pad 13: unconnected-(U3-~{DTR}-Pad13) -> CH340_DTR
- U3 pad 14: unconnected-(U3-~{RTS}-Pad14) -> CH340_RTS
- U3 pad 16: unconnected-(U3-VCC-Pad16) -> Net-(U3-V3)
- U3 pad 2: unconnected-(U3-TXD-Pad2) -> /net_lable
- U3 pad 3: unconnected-(U3-RXD-Pad3) -> /net_lable
- U3 pad 4: unconnected-(U3-V3-Pad4) -> Net-(U3-V3)
- U4 pad 1: unconnected-(U4-GND-Pad1) -> BATT_N
- U4 pad 2: unconnected-(U4-IN-Pad2) -> /3V3_LP_REG_IN
- U4 pad 3: unconnected-(U4-OUT-Pad3) -> +3V3_LP
- U5 pad 1: unconnected-(U5-STAT-Pad1) -> Net-(U5-STAT)
- U5 pad 2: unconnected-(U5-V_{SS}-Pad2) -> BATT_N
- U5 pad 3: unconnected-(U5-V_{BAT}-Pad3) -> BATT_P
- U5 pad 4: unconnected-(U5-V_{DD}-Pad4) -> Net-(D4-A)
- U5 pad 5: unconnected-(U5-PROG-Pad5) -> Net-(U5-PROG)
- U6 pad 1: unconnected-(U6-V_{DD}-Pad1) -> BATT_N
- U6 pad 2: unconnected-(U6-OUTH-Pad2) -> +3V3
- U6 pad 3: unconnected-(U6-OUTL-Pad3) -> JTAG_RST
- U7 pad 1: PWR_IN_N -> unconnected-(U7-V_{DD}-Pad1)
- U7 pad 2: +3.3V -> unconnected-(U7-OUTH-Pad2)
