File: Node/NodeHardware/NodeHardware.kicad_pcb (KiCad board)
At the start: 2 copper layers, 149 parts, among them J1 USB_C_Receptacle_16P, Q1 AO3401A, Q2 AO3401A, Q4 2N7002, Q5 2N7002, U3 CH340C, U5 MCP73831-2-OT, U8 UCC27511ADBV

Commit message: Continue schm update, slow progress
Parts:
- added C19: 100n, Capacitor_SMD:C_0805_2012Metric, F.Cu at (137.7, 57.8)
- added C38: 10u, Capacitor_SMD:C_0805_2012Metric, F.Cu at (136.8, 116.2)
- added C9: 100n, Capacitor_SMD:C_0805_2012Metric, F.Cu at (133.2, 60.8)
- added J4: PWR_IN, fflori4nComponents:TerminalBlockRemovablex2_Silk, F.Cu at (181.5, 128.2)
- added J5: BATT, fflori4nComponents:TerminalBlockRemovablex2_Silk, F.Cu at (193.0, 128.2)
- added R61: ???, Resistor_SMD:R_0805_2012Metric, F.Cu at (124.4, 72.5)
- added R70: ???, Resistor_SMD:R_0805_2012Metric, F.Cu at (128.8, 75.5)
- added U1: TPS565201DDCR, TPS565201DDCR:TPS565201DDCR_L, F.Cu at (152.0, 129.3)
- added U10: UCC27517DBVR, UCC27517DBVR:UCC27517DBVR_DBV5_TEX, F.Cu at (152.6, 102.6)
- added U11: IRLR024NTRPBF, IRLR024NTRPBF:IRLR024NTRPBF_PG-TO252-3_INF, F.Cu at (150.6, 109.4)
- added U2: SPX3819M5-L-3-3, Package_TO_SOT_SMD:SOT-23-5, F.Cu at (141.2, 131.6)
- added U4: ADS1220xPW, Package_SO:TSSOP-16_4.4x5mm_P0.65mm, F.Cu at (146.5, 90.5)
- added U6: UCC27517DBVR, UCC27517DBVR:UCC27517DBVR_DBV5_TEX, F.Cu at (147.9, 102.6)
- added U7: ESP32-S3-WROOM-1, RF_Module:ESP32-S3-WROOM-1, F.Cu at (174.6, 78.4)
- added U9: SIM7000G_DEVBoard, fflori4nComponents:sim7000G_dev_board_rev3, F.Cu at (120.5, 146.8)
- C10: value 10u -> 100n
- C11: value 1u -> 100n
- D21: value 3V6 -> YELLOW; footprint Diode_SMD:D_SOD-123 -> LED_SMD:LED_1210_3225Metric
- D3: value LED -> SS14; footprint LED_SMD:LED_1210_3225Metric -> Diode_SMD:D_SMA
- D5: value 5V1 -> YELLOW; footprint Diode_SMD:D_SOD-123 -> LED_SMD:LED_1210_3225Metric
- R10: value ??? -> 47k
- R11: value INF -> 47k
- R12: value 4k7 -> 47k
- R15: value 10k -> 0R
- R26: value 47k -> 10k
- R28: value 10K -> 10k; footprint Resistor_SMD:R_0805_2012Metric_Pad1.20x1.40mm_HandSolder -> Resistor_SMD:R_0805_2012Metric
- R30, R31: value 10K -> 47k; footprint Resistor_SMD:R_0805_2012Metric_Pad1.20x1.40mm_HandSolder -> Resistor_SMD:R_0805_2012Metric
- R33, R34, R35, R36, R38, R39: value 2k2 -> 10k
- R37: value 2k2 -> 10kk
- R48, R49, R52, R56: value 220k -> 470R
- R9: value 10k -> 47k
- TP7: value 3V3_TP -> 3V3_Bypass_TP
- TP8: value 3V3_LP_TP -> 3V3_TP
- U8: value UCC27511ADBV -> IRLR024NTRPBF; footprint Package_TO_SOT_SMD:SOT-23-6 -> IRLR024NTRPBF:IRLR024NTRPBF_PG-TO252-3_INF
- moved Q1 75.0 mm to (118.7, 130.8)
- moved Q2 75.0 mm to (118.7, 135.4)
- moved J1 75.0 mm to (110.4, 133.8)
- moved R22 73.4 mm to (115.6, 118.8)
- moved R15 71.4 mm to (111.2, 115.9)
- moved R16 71.4 mm to (111.2, 118.8)
- moved TP3 66.8 mm to (110.6, 122.3)
- moved TP4 66.8 mm to (110.6, 126.4)
- moved TP7 66.8 mm to (118.7, 122.3)
- moved TP8 66.8 mm to (118.7, 126.4)
- moved TP1 66.8 mm to (106.6, 122.3)
- moved TP2 66.8 mm to (106.6, 126.4)
- moved TP5 66.8 mm to (114.7, 122.3)
- moved TP6 66.8 mm to (114.7, 126.4)
- moved R26 62.8 mm to (106.8, 69.5)
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Connections:
- net /MCU_And_Peripherals/UART_RX_LED_K renamed /MCU_And_Peripherals/UART0_RX_LED_K
- net /MCU_And_Peripherals/UART_TX_LED_K renamed /MCU_And_Peripherals/UART0_TX_LED_K
- net 5V_REG_EN renamed Net-(U1-EN)
- net UART_UC_RX renamed UART0_UC_RX
- net UART_UC_TX renamed UART0_UC_TX
- C10 pad 1: +3V3 -> 5V_SENSE
- C11 pad 1: +3V3 -> PWR_SENSE
- C14 pad 1: +3V3_LP -> +3V3
- C23 pad 1: BATT_SENSE -> BATT_N
- C23 pad 2: BATT_N -> +3V3
- C8 pad 1: /3V3_REG_SW -> BATT_SENSE
- C8 pad 2: Net-(U2-VBST) -> BATT_N
- D21 pad 1: /MCU_And_Peripherals/AIN_1 -> /MCU_And_Peripherals/UART1_TX_LED_K
- D21 pad 2: BATT_N -> +3V3
- D3 pad 1: /3V3_REG_LED_K -> +BATT
- D3 pad 2: +3V3 -> BATT_P
- D5 pad 1: +BATT -> /MCU_And_Peripherals/UART1_RX_LED_K
- D5 pad 2: /BATT_IN_ZENER -> +3V3
- Q2 pad 1: /BATT_IN_ZENER -> BATT_N
- R10 pad 1: +3V3 -> BATT_SENSE
- R10 pad 2: /3V3_REG_VFB -> BATT_N
- R11 pad 1: BATT_N -> +3V3
- R11 pad 2: 3V3_REG_EN -> 3V3_SENSE
- R12 pad 1: /3V3_REG_LED_K -> 3V3_SENSE
- R15 pad 1: /3V3_REG_VFB -> +5V
- R15 pad 2: BATT_N -> /3V3_LP_REG_IN
- R17 pad 1: /net_lable -> /CH340_TX
- R19 pad 1: /net_lable -> /CH340_RX
- R26 pad 1: /BATT_IN_ZENER -> /MCU_And_Peripherals/UART1_RX_LED_K
- R26 pad 2: BATT_N -> UART1_UC_RX
- R28 pad 1: /MCU_And_Peripherals/GSM_PWR_KEY -> /MCU_And_Peripherals/UART1_TX_LED_K
- R28 pad 2: +5V -> UART1_UC_TX
- R30 pad 1: unconnected-(R30-Pad1) -> +5V
- R30 pad 2: unconnected-(R30-Pad2) -> 5V_SENSE
- R31 pad 1: unconnected-(R31-Pad1) -> 5V_SENSE
- R31 pad 2: unconnected-(R31-Pad2) -> BATT_N
- R45 pad 1: +BATT -> V_IN
- R45 pad 2: BATT_SENSE -> PWR_SENSE
- R47 pad 1: BATT_SENSE -> PWR_SENSE
- R8 pad 1: +5V -> Net-(U2-EN)
- R8 pad 2: /3V3_REG_IN -> /3V3_LP_REG_IN
- R9 pad 1: /3V3_REG_IN -> +BATT
- R9 pad 2: 3V3_REG_EN -> BATT_SENSE
- TP7 pad 1: +3V3 -> Net-(U2-BP)
- TP8 pad 1: +3V3_LP -> +3V3
- U3 pad 2: /net_lable -> /CH340_TX
- U3 pad 3: /net_lable -> /CH340_RX
- U8 pad 1: unconnected-(U8-V_{DD}-Pad1) -> Net-(U8-G)
- U8 pad 2: unconnected-(U8-OUTH-Pad2) -> DIG_OUT_01
- U8 pad 3: unconnected-(U8-OUTL-Pad3) -> BATT_N
Other:
- board outline added: 100 x 100 mm

Commit message: Never ending SCHM design
Parts:
- removed C1, C10, C11, C12, C15, C18, C19, C23, C24, C25, C26, C27, C28, C29, C31, C32, C33, C34, C35, C8, C9: 100n, Capacitor_SMD:C_0805_2012Metric
- removed C13, C16: 4u7, Capacitor_SMD:C_0805_2012Metric
- removed C14, C17, C4, C7: 1u, Capacitor_SMD:C_0805_2012Metric
- removed C20, C21, C22: C, Capacitor_SMD:C_0805_2012Metric
- removed C3, C38, C6: 10u, Capacitor_SMD:C_0805_2012Metric
- removed D1: LED, LED_SMD:LED_1210_3225Metric
- removed D10, D11, D12, D21, D5, D8, D9: YELLOW, LED_SMD:LED_1210_3225Metric
- removed D13, D14, D22, D23: 3V6, Diode_SMD:D_SOD-123
- removed D15, D16, D17, D18, D19, D20, D24, D25, D26, D27, D28, D29: SS34, Diode_SMD:D_SMA
- removed D2: 5V1, Diode_SMD:D_SOD-123
- removed D3: SS14, Diode_SMD:D_SMA
- removed D4: BLUE, LED_SMD:LED_1210_3225Metric
- removed D6: RED, LED_SMD:LED_1210_3225Metric
- removed D7: GREEN, LED_SMD:LED_1210_3225Metric
- removed H1, H2, H3, H4: MountingHole, MountingHole:MountingHole_3.2mm_M3_Pad_Via
- removed J1: USB_C_Receptacle_16P, Connector_USB:USB_C_Receptacle_G-Switch_GT-USB-7010ASV
- removed J4: PWR_IN, fflori4nComponents:TerminalBlockRemovablex2_Silk
- removed J5: BATT, fflori4nComponents:TerminalBlockRemovablex2_Silk
- removed Q1, Q2: AO3401A, Package_TO_SOT_SMD:SOT-23
- removed Q4, Q5: 2N7002, Package_TO_SOT_SMD:SOT-23
- removed R1, R13, R14, R15, R17, R19, R20, R21, R22, R24, R25, R29, R32, R8: 0R, Resistor_SMD:R_0805_2012Metric
- removed R10, R11, R12, R27, R30, R31, R45, R46, R47, R5, R9: 47k, Resistor_SMD:R_0805_2012Metric
- removed R16, R18: 5k1, Resistor_SMD:R_0805_2012Metric
- removed R2, R26, R28, R33, R34, R35, R36, R38, R39, R41, R42, R43, R58, R59, R60, R67, R68, R69, R7, TH1: 10k, Resistor_SMD:R_0805_2012Metric
- removed R23, R40, R44: 2k2, Resistor_SMD:R_0805_2012Metric
- removed R3: 54.9k, Resistor_SMD:R_0805_2012Metric
- removed R37: 10kk, Resistor_SMD:R_0805_2012Metric
- removed R4: INF, Resistor_SMD:R_0805_2012Metric
- removed R48, R49, R52, R56: 470R, Resistor_SMD:R_0805_2012Metric
- removed R50, R51, R62, R63: 100k, Resistor_SMD:R_0805_2012Metric
- removed R53, R54, R55, R64, R65, R66: 100R, Resistor_SMD:R_0805_2012Metric
- removed R6: 4k7, Resistor_SMD:R_0805_2012Metric
- removed R61, R70: ???, Resistor_SMD:R_0805_2012Metric
- removed TP1: V_IN_TP, TestPoint:TestPoint_Pad_D2.0mm
- removed TP10, TP9: TestPoint, TestPoint:TestPoint_Pad_D2.0mm
- removed TP2: 5V_TP, TestPoint:TestPoint_Pad_D2.0mm
- removed TP3: GND_TP_1, TestPoint:TestPoint_Pad_D2.0mm
- removed TP4: GND_TP_2, TestPoint:TestPoint_Pad_D2.0mm
- removed TP5: GND_TP_3, TestPoint:TestPoint_Pad_D2.0mm
- removed TP6: GND_TP_4, TestPoint:TestPoint_Pad_D2.0mm
- removed TP7: 3V3_Bypass_TP, TestPoint:TestPoint_Pad_D2.0mm
- removed TP8: 3V3_TP, TestPoint:TestPoint_Pad_D2.0mm
- removed U1: TPS565201DDCR, TPS565201DDCR:TPS565201DDCR_L
- removed U10, U6: UCC27517DBVR, UCC27517DBVR:UCC27517DBVR_DBV5_TEX
- removed U11, U8: IRLR024NTRPBF, IRLR024NTRPBF:IRLR024NTRPBF_PG-TO252-3_INF
- removed U2: SPX3819M5-L-3-3, Package_TO_SOT_SMD:SOT-23-5
- removed U3: CH340C, Package_SO:SOIC-16_3.9x9.9mm_P1.27mm
- removed U4: ADS1220xPW, Package_SO:TSSOP-16_4.4x5mm_P0.65mm
- removed U5: MCP73831-2-OT, Package_TO_SOT_SMD:SOT-23-5
- removed U7: ESP32-S3-WROOM-1, RF_Module:ESP32-S3-WROOM-1
- removed U9: SIM7000G_DEVBoard, fflori4nComponents:sim7000G_dev_board_rev3

Commit message: Halfway working on PCB for Node
Parts:
- added C1: 100u, Capacitor_SMD:CP_Elec_6.3x7.7, F.Cu at (-136.3, 42.0)
- added C10: 1u, Capacitor_SMD:C_0805_2012Metric, F.Cu at (-86.7, 40.3)
- added C11: 1u, Capacitor_SMD:C_0805_2012Metric, F.Cu at (-179.1, 96.6)
- added C12: 100n, Capacitor_SMD:C_0805_2012Metric, F.Cu at (329.6, 72.2)
- added C13: 470u, Capacitor_SMD:CP_Elec_6.3x7.7, F.Cu at (-103.7, -43.1)
- added C14: 100u, Capacitor_SMD:CP_Elec_6.3x7.7, F.Cu at (-103.7, -35.0)
- added C15: 10u, Capacitor_SMD:C_0805_2012Metric, F.Cu at (-102.2, -17.4)
- added C16: 100n, Capacitor_SMD:C_0805_2012Metric, F.Cu at (-56.8, 233.5)
- added C17: 100n, Capacitor_SMD:C_0805_2012Metric, F.Cu at (-56.8, 236.5)
- added C18: 22u, Capacitor_SMD:C_0805_2012Metric, F.Cu at (341.4, 61.6)
- added C19: 100n, Capacitor_SMD:C_0805_2012Metric, F.Cu at (339.1, 61.6)
- added C2: 10u, Capacitor_SMD:C_0805_2012Metric, F.Cu at (-91.2, 37.3)
- added C20: 100n, Capacitor_SMD:C_0805_2012Metric, F.Cu at (-56.8, 245.6)
- added C21: 100n, Capacitor_SMD:C_0805_2012Metric, F.Cu at (-56.8, 248.6)
- added C22: 100n, Capacitor_SMD:C_0805_2012Metric, F.Cu at (-56.8, 251.6)
- added C23: 100n, Capacitor_SMD:C_0805_2012Metric, F.Cu at (-52.4, 233.5)
- added C24: 100n, Capacitor_SMD:C_0805_2012Metric, F.Cu at (166.0, 253.1)
- added C25: 100n, Capacitor_SMD:C_0805_2012Metric, F.Cu at (380.9, 71.2)
- added C28: 1u, Capacitor_SMD:C_0805_2012Metric, F.Cu at (335.4, 74.6)
- added C29: 100n, Capacitor_SMD:C_0805_2012Metric, F.Cu at (335.4, 72.4)
- added C3: 4u7, Capacitor_SMD:C_0805_2012Metric, F.Cu at (-183.5, 93.6)
- added C30: 100n, Capacitor_SMD:C_0805_2012Metric, F.Cu at (379.2, 74.2)
- added C31: C, Capacitor_SMD:C_0805_2012Metric, F.Cu at (362.8, 84.6)
- added C32: 100n, Capacitor_SMD:C_0805_2012Metric, F.Cu at (143.1, 272.0)
- added C33: 100n, Capacitor_SMD:C_0805_2012Metric, F.Cu at (143.1, 275.0)
- added C34: 100n, Capacitor_SMD:C_0805_2012Metric, F.Cu at (371.7, 78.0)
- added C35: 100n, Capacitor_SMD:C_0805_2012Metric, F.Cu at (371.7, 74.2)
- added C36: 100n, Capacitor_SMD:C_0805_2012Metric, F.Cu at (346.8, 84.6)
- added C37: 100n, Capacitor_SMD:C_0805_2012Metric, F.Cu at (150.1, 269.0)
- added C38: 100n, Capacitor_SMD:C_0805_2012Metric, F.Cu at (150.1, 272.0)
- added C39: 100n, Capacitor_SMD:C_0805_2012Metric, F.Cu at (379.2, 78.0)
- added C4: 1u, Capacitor_SMD:C_0805_2012Metric, F.Cu at (-91.2, 43.3)
- added C5: 4u7, Capacitor_SMD:C_0805_2012Metric, F.Cu at (-183.5, 99.6)
- added C6: 100n, Capacitor_SMD:C_0805_2012Metric, F.Cu at (-183.5, 102.6)
- added C7: 100n, Capacitor_SMD:C_0805_2012Metric, F.Cu at (-91.2, 52.4)
- added C8: 100u, Capacitor_SMD:CP_Elec_6.3x7.7, F.Cu at (-136.3, 50.2)
- added C9: 10u, Capacitor_SMD:C_0805_2012Metric, F.Cu at (-86.7, 37.3)
- added D1: SS14, Diode_SMD:D_SMA, F.Cu at (-203.8, 89.6)
- added D10: BAT54S, Package_TO_SOT_SMD:SOT-23, F.Cu at (-74.3, 258.4)
- added D11: RED, LED_SMD:LED_1210_3225Metric, F.Cu at (44.7, 75.1)
- added D12: GREEN, LED_SMD:LED_1210_3225Metric, F.Cu at (44.7, 79.4)
- added D13: YELLOW, LED_SMD:LED_1210_3225Metric, F.Cu at (44.7, 83.7)
- added D14: YELLOW, LED_SMD:LED_1210_3225Metric, F.Cu at (44.7, 88.0)
- added D15: YELLOW, LED_SMD:LED_1210_3225Metric, F.Cu at (44.7, 92.3)
- added D16: YELLOW, LED_SMD:LED_1210_3225Metric, F.Cu at (50.3, 75.1)
- added D17: 3V6, Diode_SMD:D_SOD-123, F.Cu at (156.5, 253.3)
- added D18: 3V6, Diode_SMD:D_SOD-123, F.Cu at (156.5, 256.7)
- added D19: YELLOW, LED_SMD:LED_1210_3225Metric, F.Cu at (50.3, 79.4)
- added D2: 3v3, Diode_SMD:D_SOD-123, F.Cu at (-112.4, 35.7)
- added D20: YELLOW, LED_SMD:LED_1210_3225Metric, F.Cu at (50.3, 83.7)
- added D21: 3V6, Diode_SMD:D_SOD-123, F.Cu at (156.5, 260.0)
- added D22: 3V6, Diode_SMD:D_SOD-123, F.Cu at (156.5, 263.4)
- added D23: YELLOW, LED_SMD:LED_1210_3225Metric, F.Cu at (50.3, 88.0)
- added D24: YELLOW, LED_SMD:LED_1210_3225Metric, F.Cu at (50.3, 92.3)
- added D25: YELLOW, LED_SMD:LED_1210_3225Metric, F.Cu at (56.0, 75.1)
- added D26: YELLOW, LED_SMD:LED_1210_3225Metric, F.Cu at (56.0, 79.4)
- added D27: YELLOW, LED_SMD:LED_1210_3225Metric, F.Cu at (56.0, 83.7)
- added D3: BLUE, LED_SMD:LED_1210_3225Metric, F.Cu at (-221.5, 84.6)
- added D4: LED, LED_SMD:LED_1210_3225Metric, F.Cu at (-129.0, 31.0)
- added D5: BAT54S, Package_TO_SOT_SMD:SOT-23, F.Cu at (-79.2, 258.4)
- added D6: BAT54S, Package_TO_SOT_SMD:SOT-23, F.Cu at (-77.5, 233.6)
- added D7: BAT54S, Package_TO_SOT_SMD:SOT-23, F.Cu at (-77.5, 238.2)
- added D8: BAT54S, Package_TO_SOT_SMD:SOT-23, F.Cu at (-77.5, 242.8)
- added D9: BAT54S, Package_TO_SOT_SMD:SOT-23, F.Cu at (-77.5, 247.4)
- added G***: LOGO, node_logo:node_logo, F.Cu at (391.1, 67.4)
- added H1: MountingHole, MountingHole:MountingHole_3.2mm_M3_Pad_Via, F.Cu at (311.6, 58.1)
- added H2: MountingHole, MountingHole:MountingHole_3.2mm_M3_Pad_Via, F.Cu at (401.6, 58.1)
- added H3: MountingHole, MountingHole:MountingHole_3.2mm_M3_Pad_Via, F.Cu at (311.6, 148.1)
- added H4: MountingHole, MountingHole:MountingHole_3.2mm_M3_Pad_Via, F.Cu at (401.6, 148.1)
- added J1: PWR_OUT_5V, TerminalBlock:TerminalBlock_bornier-6_P5.08mm, F.Cu at (-121.2, 98.0)
- added J10: PWR_OUT_GND, TerminalBlock:TerminalBlock_bornier-4_P5.08mm, F.Cu at (-120.6, 126.5)
- added J11: DIG_IO_04, TerminalBlock:TerminalBlock_bornier-2_P5.08mm, F.Cu at (370.4, 158.6)
- added J12: DIG_IO_05, TerminalBlock:TerminalBlock_bornier-2_P5.08mm, F.Cu at (381.1, 158.6)
- added J13: DIG_IO_06, TerminalBlock:TerminalBlock_bornier-2_P5.08mm, F.Cu at (391.6, 158.6)
- added J14: ANA_IN_01, TerminalBlock:TerminalBlock_bornier-2_P5.08mm, F.Cu at (78.0, 256.0)
- added J15: ANA_IN_01, TerminalBlock:TerminalBlock_bornier-2_P5.08mm, F.Cu at (103.0, 255.5)
- added J16: ANA_IN_01, TerminalBlock:TerminalBlock_bornier-2_P5.08mm, F.Cu at (103.0, 264.6)
- added J17: ANA_IN_01, TerminalBlock:TerminalBlock_bornier-2_P5.08mm, F.Cu at (89.5, 256.0)
- added J18: CONN_I2C, TerminalBlock:TerminalBlock_bornier-4_P5.08mm, F.Cu at (-203.7, 161.0)
- added J19: CONN_SPI, TerminalBlock:TerminalBlock_bornier-6_P5.08mm, F.Cu at (-173.7, 161.0)
- added J2: PWR_OUT_3V3, TerminalBlock:TerminalBlock_bornier-6_P5.08mm, F.Cu at (-121.8, 112.5)
- added J20: DIG_OUT_01, TerminalBlock:TerminalBlock_bornier-2_P5.08mm, F.Cu at (317.9, 158.6)
- added J21: DIG_OUT_02, TerminalBlock:TerminalBlock_bornier-2_P5.08mm, F.Cu at (328.1, 158.6)
- added J3: PWR_IN, fflori4nComponents:TerminalBlockRemovablex2, F.Cu at (-161.8, 39.5)
- added J4: BATT, fflori4nComponents:TerminalBlockRemovablex2, F.Cu at (-271.5, 89.9)
- added J5: USB_C_Receptacle_16P, Connector_USB:USB_C_Receptacle_G-Switch_GT-USB-7010ASV, F.Cu at (322.4, 57.4)
- added J6: DIG_IO_01, TerminalBlock:TerminalBlock_bornier-2_P5.08mm, F.Cu at (338.6, 158.6)
- added J7: DIG_IO_02, TerminalBlock:TerminalBlock_bornier-2_P5.08mm, F.Cu at (349.2, 158.6)
- added J8: DIG_IO_03, TerminalBlock:TerminalBlock_bornier-2_P5.08mm, F.Cu at (359.9, 158.6)
- added J9: ESP32_JTAG, Connector_PinHeader_2.54mm:PinHeader_1x07_P2.54mm_Vertical, F.Cu at (380.1, 58.1)
- added L1: 3.3uH, Inductor_SMD:L_6.3x6.3_H3, F.Cu at (-119.6, 33.4)
- added N1: Housing, PlasticEnclosures:PlasticEnclosure_150x110x70, F.Cu at (150.0, 100.0)
- added Q1: AO3401A, Package_TO_SOT_SMD:SOT-23, F.Cu at (-98.9, 42.8)
- added Q2: AO3401A, Package_TO_SOT_SMD:SOT-23, F.Cu at (-191.3, 100.7)
- added Q3: AO3400A, Package_TO_SOT_SMD:SOT-23, F.Cu at (-72.6, 233.6)
- added Q4: AO3400A, Package_TO_SOT_SMD:SOT-23, F.Cu at (-72.6, 238.2)
- added Q5: 2N7002, Package_TO_SOT_SMD:SOT-23, F.Cu at (328.1, 78.0)
- added Q6: 2N7002, Package_TO_SOT_SMD:SOT-23, F.Cu at (321.7, 78.0)
- added R1: 47k, Resistor_SMD:R_0805_2012Metric, F.Cu at (-127.0, 44.4)
- added R10: 0R, Resistor_SMD:R_0805_2012Metric, F.Cu at (-222.8, 109.9)
- added R11: 54.9k, Resistor_SMD:R_0805_2012Metric, F.Cu at (-122.5, 56.2)
- added R12: 10k, Resistor_SMD:R_0805_2012Metric, F.Cu at (-122.5, 59.1)
- added R13: 0R, Resistor_SMD:R_0805_2012Metric, F.Cu at (-218.4, 101.1)
- added R14: 0R, Resistor_SMD:R_0805_2012Metric, F.Cu at (-118.1, 47.3)
- added R15: 4k7, Resistor_SMD:R_0805_2012Metric, F.Cu at (-118.1, 50.3)
- added R16: 5k1, Resistor_SMD:R_0805_2012Metric, F.Cu at (326.4, 65.2)
- added R17: 5k1, Resistor_SMD:R_0805_2012Metric, F.Cu at (319.6, 65.2)
- added R18: 0R, Resistor_SMD:R_0805_2012Metric, F.Cu at (317.4, 65.2)
- added R19: 0R, Resistor_SMD:R_0805_2012Metric, F.Cu at (324.1, 65.2)
- added R2: 2k2, Resistor_SMD:R_0805_2012Metric, F.Cu at (-227.2, 104.0)
- added R20: 0R, Resistor_SMD:R_0805_2012Metric, F.Cu at (321.9, 65.2)
- added R21: 0R, Resistor_SMD:R_0805_2012Metric, F.Cu at (329.6, 74.7)
- added R22: 0R, Resistor_SMD:R_0805_2012Metric, F.Cu at (329.6, 69.7)
- added R23: 0R, Resistor_SMD:R_0805_2012Metric, F.Cu at (329.6, 67.4)
- added R24: 10k, Resistor_SMD:R_0805_2012Metric, F.Cu at (-90.6, 235.5)
- added R25: 10k, Resistor_SMD:R_0805_2012Metric, F.Cu at (-90.6, 238.4)
- added R26: 220R, Resistor_SMD:R_0805_2012Metric, F.Cu at (-90.6, 241.4)
- added R27: 220R, Resistor_SMD:R_0805_2012Metric, F.Cu at (-90.6, 244.3)
- added R28: 100R, Resistor_SMD:R_0805_2012Metric, F.Cu at (-90.6, 247.3)
- added R29: 100R, Resistor_SMD:R_0805_2012Metric, F.Cu at (-90.6, 250.2)
- added R3: 0R, Resistor_SMD:R_0805_2012Metric, F.Cu at (-127.0, 50.3)
- added R30: 10k, Resistor_SMD:R_0805_2012Metric, F.Cu at (-90.6, 253.2)
- added R31: 10k, Resistor_SMD:R_0805_2012Metric, F.Cu at (-90.6, 256.1)
- added R32: 220R, Resistor_SMD:R_0805_2012Metric, F.Cu at (-90.6, 259.1)
- added R33: 220R, Resistor_SMD:R_0805_2012Metric, F.Cu at (-90.6, 262.1)
- added R34: 100R, Resistor_SMD:R_0805_2012Metric, F.Cu at (-86.2, 235.5)
- added R35: 100R, Resistor_SMD:R_0805_2012Metric, F.Cu at (-86.2, 238.4)
- added R36: 0R, Resistor_SMD:R_0805_2012Metric, F.Cu at (329.6, 65.2)
- added R37: 0R, Resistor_SMD:R_0805_2012Metric, F.Cu at (329.6, 62.9)
- added R38: 10k, Resistor_SMD:R_0805_2012Metric, F.Cu at (-86.2, 247.3)
- added R39: 10k, Resistor_SMD:R_0805_2012Metric, F.Cu at (-86.2, 250.2)
- added R4: 0R, Resistor_SMD:R_0805_2012Metric, F.Cu at (-227.2, 109.9)
- added R40: 100R, Resistor_SMD:R_0805_2012Metric, F.Cu at (-86.2, 253.2)
- added R41: 100R, Resistor_SMD:R_0805_2012Metric, F.Cu at (-86.2, 256.1)
- added R42: 10k, Resistor_SMD:R_0805_2012Metric, F.Cu at (1.17, 98.1)
- added R43: 10k, Resistor_SMD:R_0805_2012Metric, F.Cu at (1.17, 101.0)
- added R44: 2k2, Resistor_SMD:R_0805_2012Metric, F.Cu at (318.4, 78.0)
- added R45: 2k2, Resistor_SMD:R_0805_2012Metric, F.Cu at (324.9, 78.0)
- added R46: 10k, Resistor_SMD:R_0805_2012Metric, F.Cu at (5.58, 80.4)
- added R47: 10k, Resistor_SMD:R_0805_2012Metric, F.Cu at (5.58, 83.3)
- added R48: 47R, Resistor_SMD:R_0805_2012Metric, F.Cu at (369.2, 66.5)
- added R49: 47R, Resistor_SMD:R_0805_2012Metric, F.Cu at (380.9, 66.7)
- added R5: 10k, Resistor_SMD:R_0805_2012Metric, F.Cu at (-127.0, 56.2)
- added R50: 47R, Resistor_SMD:R_0805_2012Metric, F.Cu at (380.9, 69.0)
- added R51: 47R, Resistor_SMD:R_0805_2012Metric, F.Cu at (369.2, 70.2)
- added R52: 47R, Resistor_SMD:R_0805_2012Metric, F.Cu at (161.6, 253.1)
- added R53: 47R, Resistor_SMD:R_0805_2012Metric, F.Cu at (161.6, 256.1)
- added R54: 47R, Resistor_SMD:R_0805_2012Metric, F.Cu at (161.6, 259.0)
- added R55: 47R, Resistor_SMD:R_0805_2012Metric, F.Cu at (161.6, 262.0)
- added R56: 10k, Resistor_SMD:R_0805_2012Metric, F.Cu at (339.5, 74.6)
- added R57: 10k, Resistor_SMD:R_0805_2012Metric, F.Cu at (9.99, 83.3)
- added R58: 2k2, Resistor_SMD:R_0805_2012Metric, F.Cu at (339.5, 72.4)
- added R59: 10k, Resistor_SMD:R_0805_2012Metric, F.Cu at (9.99, 89.2)
- added R6: INF, Resistor_SMD:R_0805_2012Metric, F.Cu at (-127.0, 59.1)
- added R60: 10k, Resistor_SMD:R_0805_2012Metric, F.Cu at (358.8, 84.6)
- added R61: 47k, Resistor_SMD:R_0805_2012Metric, F.Cu at (376.7, 74.2)
- added R62: 47k, Resistor_SMD:R_0805_2012Metric, F.Cu at (376.7, 78.0)
- added R63: 10k, Resistor_SMD:R_0805_2012Metric, F.Cu at (9.99, 101.0)
- added R64: 10k, Resistor_SMD:R_0805_2012Metric, F.Cu at (14.4, 74.5)
- added R65: 470R, Resistor_SMD:R_0805_2012Metric, F.Cu at (125.0, 260.0)
- added R66: 100k, Resistor_SMD:R_0805_2012Metric, F.Cu at (125.0, 262.9)
- added R67: 470R, Resistor_SMD:R_0805_2012Metric, F.Cu at (125.0, 265.9)
- added R68: 100k, Resistor_SMD:R_0805_2012Metric, F.Cu at (125.0, 268.9)
- added R69: 47k, Resistor_SMD:R_0805_2012Metric, F.Cu at (374.2, 74.2)
- added R7: 0R, Resistor_SMD:R_0805_2012Metric, F.Cu at (-222.8, 101.1)
- added R70: 47k, Resistor_SMD:R_0805_2012Metric, F.Cu at (374.2, 78.0)
- added R71: 47k, Resistor_SMD:R_0805_2012Metric, F.Cu at (369.2, 74.2)
- added R72: 47k, Resistor_SMD:R_0805_2012Metric, F.Cu at (369.2, 78.0)
- added R73: 10k, Resistor_SMD:R_0805_2012Metric, F.Cu at (342.9, 84.6)
- added R74: 10k, Resistor_SMD:R_0805_2012Metric, F.Cu at (18.8, 74.5)
- added R75: 470R, Resistor_SMD:R_0805_2012Metric, F.Cu at (129.5, 260.0)
- added R76: 100k, Resistor_SMD:R_0805_2012Metric, F.Cu at (129.5, 262.9)
- added R77: 470R, Resistor_SMD:R_0805_2012Metric, F.Cu at (129.5, 265.9)
- added R78: 100k, Resistor_SMD:R_0805_2012Metric, F.Cu at (129.5, 268.9)
- added R79: 47k, Resistor_SMD:R_0805_2012Metric, F.Cu at (381.7, 74.2)
- added R8: 47k, Resistor_SMD:R_0805_2012Metric, F.Cu at (-222.8, 104.0)
- added R80: 10k, Resistor_SMD:R_0805_2012Metric, F.Cu at (18.8, 92.2)
- added R9: 0R, Resistor_SMD:R_0805_2012Metric, F.Cu at (-222.8, 107.0)
- added SW1: RST, Button_Switch_SMD:SW_Push_1P1T_NO_6x6mm_H9.5mm, F.Cu at (337.4, 67.4)
- added SW2: BOOT, Button_Switch_SMD:SW_Push_1P1T_NO_6x6mm_H9.5mm, F.Cu at (360.7, 89.4)
- added SW3: BTN, Button_Switch_SMD:SW_Push_1P1T_NO_6x6mm_H9.5mm, F.Cu at (344.9, 89.4)
- added TH1: 10k, Resistor_SMD:R_0805_2012Metric, F.Cu at (381.7, 78.0)
- added TP1: V_IN_TP, TestPoint:TestPoint_Pad_D2.0mm, F.Cu at (-109.5, 44.9)
- added TP11: TP_BATT_PROT, TestPoint:TestPoint_Pad_D2.0mm, F.Cu at (-201.7, 101.6)
- added TP12: TP_3V3, TestPoint:TestPoint_Pad_D2.0mm, F.Cu at (-201.7, 105.7)
- added TP13: TP_5V, TestPoint:TestPoint_Pad_D2.0mm, F.Cu at (-101.4, 53.0)
- added TP14: TP_UART0_RX, TestPoint:TestPoint_Pad_D1.0mm, F.Cu at (156.8, -68.9)
- added TP15: TP_UART0_TX, TestPoint:TestPoint_Pad_D1.0mm, F.Cu at (156.8, -65.9)
- added TP16: TP_I2C_SCL, TestPoint:TestPoint_Pad_D1.0mm, F.Cu at (156.8, -62.8)
- added TP17: TP_I2C_SDA, TestPoint:TestPoint_Pad_D1.0mm, F.Cu at (156.8, -59.8)
- added TP18: TP_DIGOUT_01, TestPoint:TestPoint_Pad_D1.0mm, F.Cu at (156.8, -56.7)
- added TP19: TP_DIGOUT_02, TestPoint:TestPoint_Pad_D1.0mm, F.Cu at (156.8, -53.7)
- added TP2: 3V3_Bypass_TP, TestPoint:TestPoint_Pad_D2.0mm, F.Cu at (-209.8, 105.7)
- added TP20: TP_SPI_CS_0, TestPoint:TestPoint_Pad_D1.0mm, F.Cu at (159.8, -68.9)
- added TP21: TP_SPI_CS_1, TestPoint:TestPoint_Pad_D1.0mm, F.Cu at (159.8, -65.9)
- added TP22: TP_SPI_MOSI, TestPoint:TestPoint_Pad_D1.0mm, F.Cu at (159.8, -62.8)
- added TP23: TP_SPI_SCLK, TestPoint:TestPoint_Pad_D1.0mm, F.Cu at (159.8, -59.8)
- added TP24: TP_SPI_MISO, TestPoint:TestPoint_Pad_D1.0mm, F.Cu at (159.8, -56.7)
- added TP25: TP_SPI_CS_EXT, TestPoint:TestPoint_Pad_D1.0mm, F.Cu at (159.8, -53.7)
- added TP26: TP_DIG_IO_06, TestPoint:TestPoint_Pad_D1.0mm, F.Cu at (162.9, -68.9)
- added TP27: TP_DIG_IO_05, TestPoint:TestPoint_Pad_D1.0mm, F.Cu at (162.9, -65.9)
- added TP28: TP_DIG_IO_04, TestPoint:TestPoint_Pad_D1.0mm, F.Cu at (162.9, -62.8)
- added TP29: TP_DIG_IO_03, TestPoint:TestPoint_Pad_D1.0mm, F.Cu at (162.9, -59.8)
- added TP3: 5V_TP, TestPoint:TestPoint_Pad_D2.0mm, F.Cu at (-109.5, 53.0)
- added TP30: TP_DIG_IO_02, TestPoint:TestPoint_Pad_D1.0mm, F.Cu at (162.9, -56.7)
- added TP31: TP_DIG_IO_01, TestPoint:TestPoint_Pad_D1.0mm, F.Cu at (162.9, -53.7)
- added TP32: TP_UART1_TX, TestPoint:TestPoint_Pad_D1.0mm, F.Cu at (165.9, -68.9)
- added TP33: TP_UART1_RX, TestPoint:TestPoint_Pad_D1.0mm, F.Cu at (165.9, -65.9)
- added TP34: TP_GPIO6, TestPoint:TestPoint_Pad_D1.0mm, F.Cu at (165.9, -62.8)
- added TP35: TP_GPIO7, TestPoint:TestPoint_Pad_D1.0mm, F.Cu at (165.9, -59.8)
- added TP36: TP_GPIO8, TestPoint:TestPoint_Pad_D1.0mm, F.Cu at (165.9, -56.7)
- added TP37: TP_GPIO9, TestPoint:TestPoint_Pad_D1.0mm, F.Cu at (165.9, -53.7)
- added TP38: TP_GPIO10, TestPoint:TestPoint_Pad_D1.0mm, F.Cu at (169.0, -68.9)
- added TP39: TP_GPIO11, TestPoint:TestPoint_Pad_D1.0mm, F.Cu at (169.0, -65.9)
- added TP4: 3V3_TP, TestPoint:TestPoint_Pad_D2.0mm, F.Cu at (-209.8, 113.8)
- added TP40: TP_ANA_IN_01_UC, TestPoint:TestPoint_Pad_D1.0mm, F.Cu at (139.0, 256.9)
- added TP41: TP_ANA_IN_01, TestPoint:TestPoint_Pad_D1.0mm, F.Cu at (139.0, 259.9)
- added TP42: TP_ANA_IN_02_UC, TestPoint:TestPoint_Pad_D1.0mm, F.Cu at (139.0, 262.9)
- added TP43: TP_ANA_IN_02, TestPoint:TestPoint_Pad_D1.0mm, F.Cu at (139.0, 266.0)
- added TP44: TP_ANA_IN_04_UC, TestPoint:TestPoint_Pad_D1.0mm, F.Cu at (142.0, 250.8)
- added TP45: TP_ANA_IN_04, TestPoint:TestPoint_Pad_D1.0mm, F.Cu at (142.0, 253.8)
- added TP46: TP_ANA_IN_03_UC, TestPoint:TestPoint_Pad_D1.0mm, F.Cu at (142.0, 256.9)
- added TP47: TP_ANA_IN_03, TestPoint:TestPoint_Pad_D1.0mm, F.Cu at (142.0, 259.9)
- added TP49: TP_DIG_OUT_01, TestPoint:TestPoint_Pad_D1.0mm, F.Cu at (-46.3, 249.7)
- added TP5: GND_TP_1, TestPoint:TestPoint_Pad_D2.0mm, F.Cu at (21.1, 118.1)
- added TP51: TP_DIG_OUT_02, TestPoint:TestPoint_Pad_D1.0mm, F.Cu at (-46.3, 252.7)
- added TP52: TP_DIG_IO_04, TestPoint:TestPoint_Pad_D1.0mm, F.Cu at (-43.3, 237.4)
- added TP54: TP_DIG_IO_01, TestPoint:TestPoint_Pad_D1.0mm, F.Cu at (-43.3, 240.5)
- added TP55: TP_DIG_IO_02, TestPoint:TestPoint_Pad_D1.0mm, F.Cu at (-43.3, 243.6)
- added TP56: TP_DIG_IO_05, TestPoint:TestPoint_Pad_D1.0mm, F.Cu at (-43.3, 246.6)
- added TP57: TP_DIG_IO_03, TestPoint:TestPoint_Pad_D1.0mm, F.Cu at (-43.3, 249.7)
- added TP58: TP_DIG_IO_06, TestPoint:TestPoint_Pad_D1.0mm, F.Cu at (-43.3, 252.7)
- added TP6: GND_TP_2, TestPoint:TestPoint_Pad_D2.0mm, F.Cu at (21.1, 122.2)
- added TP7: GND_TP_3, TestPoint:TestPoint_Pad_D2.0mm, F.Cu at (21.1, 126.2)
- added TP8: GND_TP_4, TestPoint:TestPoint_Pad_D2.0mm, F.Cu at (21.1, 130.2)
- added U1: MCP73831-2-OT, Package_TO_SOT_SMD:SOT-23-5, F.Cu at (-236.8, 89.0)
- added U2: TPS565201DDCR, TPS565201DDCR:TPS565201DDCR_L, F.Cu at (-105.0, 31.6)
- added U3: SPX3819M5-L-3-3, Package_TO_SOT_SMD:SOT-23-5, F.Cu at (-236.8, 93.6)
- added U4: CH340C, Package_SO:SOIC-16_3.9x9.9mm_P1.27mm, F.Cu at (322.0, 71.4)
- added U5: SIM7000G_DEVBoard, fflori4nComponents:sim7000G_dev_board_rev3, F.Cu at (-82.0, -40.6)
- added U6: ESP32-S3-WROOM-1, RF_Module:ESP32-S3-WROOM-1, F.Cu at (353.1, 66.6)
- added U7: ADS1220xPW, Package_SO:TSSOP-16_4.4x5mm_P0.65mm, F.Cu at (374.7, 69.0)
- added U8: ADS1220xPW, Package_SO:TSSOP-16_4.4x5mm_P0.65mm, F.Cu at (164.1, 266.7)
Routing:
- added copper zone on B.Cu, net GND
- added copper zone on F.Cu, net GND
- added copper zone on In2.Cu, net GND
Other:
- outline, holes or cut-outs redrawn
- copper layers 2 -> 4

Commit message: Continue updating PCB (main form)
Parts:
- removed the J1 at (-121.2, 98.0)
- removed the J11 at (370.4, 158.6)
- removed the J2 at (-121.8, 112.5)
- removed J20: DIG_OUT_01, TerminalBlock:TerminalBlock_bornier-2_P5.08mm
- removed J21: DIG_OUT_02, TerminalBlock:TerminalBlock_bornier-2_P5.08mm
- removed the J6 at (338.6, 158.6)
- removed the J7 at (349.2, 158.6)
- added J14: DIG_IO_04, TerminalBlock:TerminalBlock_bornier-2_P5.08mm, F.Cu at (183.9, 77.2)
- added J16: DIG_OUT_02, TerminalBlock:TerminalBlock_bornier-2_P5.08mm, F.Cu at (183.9, 56.9)
- added J9: DIG_IO_01, TerminalBlock:TerminalBlock_bornier-2_P5.08mm, F.Cu at (183.9, 107.7)
- added TP33: TP_GPIO45, TestPoint:TestPoint_Pad_D1.0mm, F.Cu at (278.3, 61.7)
- added TP35: TP_GPIO46, TestPoint:TestPoint_Pad_D1.0mm, F.Cu at (278.3, 64.7)
- J10: value PWR_OUT_GND -> DIG_IO_03; footprint TerminalBlock:TerminalBlock_bornier-4_P5.08mm -> TerminalBlock:TerminalBlock_bornier-2_P5.08mm
- J11: renamed from J15; value ANA_IN_01 -> ANA_IN_02
- J12: value DIG_IO_05 -> PWR_OUT; footprint TerminalBlock:TerminalBlock_bornier-2_P5.08mm -> TerminalBlock:TerminalBlock_bornier-4_P5.08mm
- J13: value DIG_IO_06 -> DIG_IO_02
- J15: renamed from J16; value ANA_IN_01 -> ANA_IN_03
- J17: value ANA_IN_01 -> ANA_IN_04
- J4: renamed from J3; footprint fflori4nComponents:TerminalBlockRemovablex2 -> TerminalBlock:TerminalBlock_bornier-2_P5.08mm
- J6: renamed from J4; footprint fflori4nComponents:TerminalBlockRemovablex2 -> TerminalBlock:TerminalBlock_bornier-2_P5.08mm
- J8: value DIG_IO_03 -> DIG_OUT_01
- moved TP10 507.7 mm to (297.2, 141.0)
- moved R17 507.5 mm to (279.5, 137.1)
- moved R18 507.5 mm to (283.9, 134.1)
- moved R19 507.5 mm to (288.3, 128.2)
- moved R20 507.5 mm to (279.5, 131.2)
- moved R21 507.5 mm to (283.9, 137.1)
- moved R22 507.5 mm to (283.9, 128.2)
- moved R23 507.5 mm to (283.9, 131.2)
- moved TP11 507.5 mm to (297.0, 132.8)
- moved U4 507.0 mm to (269.4, 121.0)
- moved U5 507.0 mm to (269.4, 116.4)
- moved D3 496.2 mm to (292.3, 102.2)
- moved D4 495.5 mm to (273.9, 97.3)
- moved C13 488.6 mm to (309.0, 118.9)
- moved C12 482.5 mm to (298.7, 117.2)
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- renumbered C7 to C1, C14 to C10, C15 to C11, C5 to C12, C11 to C13, C6 to C14, C3 to C15, C18 to C16, C19 to C17, C28 to C18, C29 to C19, C1 to C2, C31 to C20, C36 to C21, C25 to C22, C30 to C23, C34 to C24, C35 to C25, C39 to C26, C32 to C27, C37 to C28, C24 to C29, C2 to C3, C16 to C30, C20 to C31, C38 to C32, C22 to C33, C17 to C34, C21 to C35, C23 to C37, C8 to C5, C9 to C6, C10 to C7, C12 to C8, C13 to C9, D2 to D1, D15 to D10, D16 to D11, D23 to D12, D11 to D13, D12 to D14, D25 to D15, D26 to D16, D27 to D17, D17 to D18, D21 to D19, D4 to D2, D5 to D20, D7 to D21, D9 to D22, D18 to D23, D6 to D24, D8 to D25, D10 to D27, D1 to D3, D3 to D4, D24 to D5, D19 to D6, D20 to D7, D13 to D8, D14 to D9, J18 to J1, J5 to J2, J19 to J3, J9 to J5, J14 to J7, Q5 to Q3, Q6 to Q4, Q3 to Q5, Q4 to Q6, R3 to R1, R21 to R10, R16 to R11, R17 to R12, R22 to R13, R23 to R14, R19 to R15, R20 to R16, R4 to R17, R9 to R18, R13 to R19, R14 to R2, R2 to R20, R10 to R21, R7 to R22, R8 to R23, R46 to R24, R47 to R25, R57 to R26, R59 to R27, R74 to R28, R42 to R29, R5 to R3, R43 to R30, R64 to R31, R36 to R32, R63 to R33, R37 to R34, R80 to R35, R44 to R36, R56 to R37, R60 to R38, R58 to R39, R11 to R4, R73 to R40, R45 to R41, R61 to R42, R69 to R43, R71 to R44, R79 to R45, R62 to R46, R70 to R47, R72 to R48, R48 to R49, R6 to R5, R26 to R50, R32 to R51, R49 to R52, R50 to R53, R27 to R54, R33 to R55, R51 to R56, R65 to R57, R75 to R58, R66 to R59, R1 to R6, R76 to R60, R77 to R61, R67 to R62, R28 to R63, R34 to R64, R24 to R65, R40 to R65, R30 to R66, R78 to R67, R52 to R69, R38 to R69, R15 to R7, R53 to R70, R54 to R71, R55 to R72, R29 to R73, R35 to R74, R25 to R75, R31 to R76, R41 to R77, R12 to R8, R39 to R80, R18 to R9, TP5 to TP1, TP4 to TP10, TP2 to TP11, TP15 to TP12, TP14 to TP13, TP20 to TP14, TP21 to TP15, TP6 to TP2, TP34 to TP20, TP35 to TP21, TP36 to TP22, TP37 to TP23, TP38 to TP24, TP39 to TP25, TP31 to TP26, TP30 to TP27, TP29 to TP28, TP32 to TP29, TP7 to TP3, TP33 to TP30, TP28 to TP31, TP27 to TP32, TP22 to TP34, TP23 to TP36, TP26 to TP37, TP24 to TP38, TP25 to TP39, TP8 to TP4, TP49 to TP40, TP51 to TP41, TP41 to TP42, TP40 to TP44, TP42 to TP45, TP45 to TP46, TP54 to TP48, TP57 to TP49, TP55 to TP49, TP1 to TP5, TP44 to TP50, TP46 to TP51, TP58 to TP53, TP56 to TP53, TP3 to TP6, TP13 to TP7, TP11 to TP8, TP12 to TP9, U2 to U1, U4 to U2, U5 to U3, U3 to U4, U1 to U5
Connections:
- C34 pad 1: DIG_IO_04_UC -> DIG_IO_03_UC
- C35 pad 1: DIG_IO_05_UC -> DIG_IO_04_UC
- D24 pad 3: DIG_IO_04_UC -> DIG_IO_03_UC
- D25 pad 3: DIG_IO_05_UC -> DIG_IO_04_UC
- J10 pad 2: GND -> DIG_IO_03
- J12 pad 2: DIG_IO_05 -> +3V3
- J13 pad 2: DIG_IO_06 -> DIG_IO_02
- J8 pad 2: DIG_IO_03 -> DIG_OUT_01
- R73 pad 1: DIG_IO_04_UC -> DIG_IO_03_UC
- R73 pad 2: DIG_IO_04 -> DIG_IO_03
- R74 pad 1: DIG_IO_05_UC -> DIG_IO_04_UC
- R74 pad 2: DIG_IO_05 -> DIG_IO_04
- R75 pad 1: DIG_IO_04_UC -> DIG_IO_03_UC
- R76 pad 1: DIG_IO_05_UC -> DIG_IO_04_UC
- TP32 pad 1: DIG_IO_05_UC -> LED_01
- TP37 pad 1: DIG_IO_06_UC -> LED_02
- TP52 pad 1: DIG_IO_04 -> DIG_IO_03
- TP53 pad 1: DIG_IO_05 -> DIG_IO_04
- U6 pad 16: LED_02 -> Net-(U6-GPIO46)
- U6 pad 24: DIG_IO_06_UC -> LED_02
- U6 pad 26: LED_01 -> Net-(U6-GPIO45)
- U6 pad 31: DIG_IO_05_UC -> LED_01
Other:
- board size 100 x 100 mm -> 80 x 106 mm
- board text added: "${REFERENCE}"
