File: Node/NodeHardware/NodeHardware.kicad_sch (KiCad schematic)
At the start: 69 parts, among them J1 USB_C_Receptacle_16P, J10 PWR_OUT_5V, J11 PWR_OUT_3V3, J3 ESP32_JTAG, J4 PWR_IN, J5 BATT, J7 DIG_IO_A, J8 DIG_IO_B, J9 ANA_IN, Q1 AO3401A, Q2 AO3401A, U1 TPS565201DDCR, U2 SPX3819M5-L-3-3, U3 CH340C, U5 MCP73831-2-OT, U9 SIM7000G_DEVBoard

Commit message: Continue updating schm for initial version
Parts:
- added J2: CONN_I2C, symbol Connector_Generic:Conn_01x04
- added J6: CONN_SPI, symbol Connector_Generic:Conn_01x07
- added R15: 0R, Resistor_SMD:R_0805_2012Metric, symbol Device:R
- TP8: value 3V3_LP_TP -> 3V3_TP
Connections:
- net +3.3V: now also J11.1 (Pin_1), J11.2 (Pin_2), J11.3 (Pin_3), J11.4 (Pin_4)
- net +3V3: now also C14.1, TP8.1, U2.5 (OUT), J2.4 (Pin_4), J6.7 (Pin_7)
- net +5V: now also R15.1
- net 3V3_LP_REG_IN: now also R15.2
- net GND: now also J2.1 (Pin_1), J6.1 (Pin_1)
- removed net +3V3_LP: C14.1, J11.1 (Pin_1), J11.2 (Pin_2), J11.3 (Pin_3), J11.4 (Pin_4), TP8.1, U2.5 (OUT)
- net UART_UC_RX renamed UART0_UC_RX
- net UART0_UC_RX: no longer U9.8 (TXD)
- net UART_UC_TX renamed UART0_UC_TX
- net UART0_UC_TX: no longer U9.6 (RXD)
- net net_lable renamed CH340_RX
- net CH340_RX: no longer R17.1, U3.2 (TXD)
- new net CH340_TX: R17.1, U3.2 (TXD)
- new net I2C_SCL: J2.2 (Pin_2)
- new net I2C_SDA: J2.3 (Pin_3)
- new net SPI_CS0: J6.5 (Pin_5)
- new net SPI_CS1: J6.6 (Pin_6)
- new net SPI_MISO: J6.4 (Pin_4)
- new net SPI_MOSI: J6.3 (Pin_3)
- new net SPI_SCLK: J6.2 (Pin_2)
- new net UART1_UC_RX: U9.8 (TXD)
- new net UART1_UC_TX: U9.6 (RXD)
- no-connect marks 9 -> 11
Other:
- note added: "Comms"
- moved on the sheet: C12, C15, D1, J1, R16, R18

Commit message: Continue schm update, slow progress
Parts:
- U9: footprint myComponents:sim7000G_dev_board_rev3 -> fflori4nComponents:sim7000G_dev_board_rev3
Connections:
- net 5V_REG_EN: no longer names the net of R2.2, R4.2, U1.5 (EN)
Changed lines of the file:
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@@
 	(wire
 		(pts
-			(xy 124.46 49.53) (xy 125.73 49.53)
-		)
-		(stroke
-			(width 0)
-			(type default)
-		)
-	)
-	(wire
-		(pts
 			(xy 38.1 62.23) (xy 50.8 62.23)
 		)
@@
 	(text_box "Is this the best way to have the option of powering the ESP with both LiIon battery and external power supply? Is there a way to make this 'switch automatically'?"
 		(exclude_from_sim no)
-		(at 146.05 137.16 0)
+		(at 146.05 130.81 0)
 		(size 22.86 12.7)
 		(stroke
@@
 		)
 	)
-	(text_box "According to the ESP32 datasheet, the power consumption \nduring RF operations in active mode is as follows:\n\nMode							Power Consumption\nWi-Fi Tx packet 13dBm~21dBm		160~260mA\nWi-Fi/BT Tx packet 0dBm			120mA\nWi-Fi/BT Rx and listeninn		80~90mA\n\nIn deep sleep mode, the chip consumes anywhere between \n0.15 mA (when the ULP coprocessor is on) and 10 µA."
+	(text_box "According to the ESP32 datasheet, the power consumption \nduring RF operations in active mode is as follows:\n\nMode							Power Consumption\nWi-Fi Tx packet 13dBm~21dBm		160~260mA\nWi-Fi/BT Tx packet 0dBm			120mA\nWi-Fi/BT Rx and listeninn		80~90mA\n\nIn deep sleep mode, the chip consumes anywhere between \n0.15 mA (when the ULP coprocessor is on) and 10 µA.\n\nIn worst case (260mA for ESP32), this leaves up to \n240mA for all other on-board devices and sensors, as \nwell as the external devices."
 		(exclude_from_sim no)
 		(at 171.45 182.88 0)
-		(size 53.7299 21.3031)
+		(size 53.7299 24.13)
 		(stroke
 			(width 0)
@@
 		)
 	)
-	(global_label "5V_REG_EN"
-		(shape input)
-		(at 124.46 49.53 180)
-		(fields_autoplaced yes)
-		(effects
-			(font
-				(size 1 1)
-			)
-			(justify right)
-		)
-		(property "Intersheetrefs" "${INTERSHEET_REFS}"
-			(at 113.9192 49.53 0)
-			(effects
-				(font
-					(size 1.27 1.27)
-				)
-				(justify right)
-				(hide yes)
-			)
-		)
-	)
 	(global_label "CH340_DTR"
 		(shape output)
@@
 		)
 		(property "Value" "+BATT"
-			(at 148.59 158.496 0)
+			(at 148.59 159.258 0)
 			(effects
 				(font
@@
 			)
 		)
-		(property "Footprint" "myComponents:sim7000G_dev_board_rev3"
+		(property "Footprint" "fflori4nComponents:sim7000G_dev_board_rev3"
 			(at 367.03 170.18 0)
 			(effects
@@
 		)
 		(property "Value" "+5V"
-			(at 148.59 151.892 0)
+			(at 148.59 152.654 0)
 			(effects
 				(font
